File: elec/modules/motordrivers/_autosave-motordrivers.kicad_sch (KiCad schematic)
At the start: 16 parts, among them IC2 VNH5019ATR-E, J1 Conn_01x02, J10 Conn_01x05, J2 Conn_01x05, J9 Conn_01x05, Q1 AON6354

Commit message: did drivers yay
Connections:
- net +3V3: now also J9.4 (Pin_4); no longer J9.3 (Pin_3)
- net M SW: now also J9.3 (Pin_3); no longer J9.4 (Pin_4)
Changed lines of the file:
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@@
 	)
 	(label "M SW"
-		(at 93.98 66.04 0)
+		(at 93.98 68.58 0)
 		(effects
 			(font
@@
 	(symbol
 		(lib_id "power:+3V3")
-		(at 93.98 68.58 270)
+		(at 93.98 66.04 270)
 		(unit 1)
 		(exclude_from_sim no)
@@
 		(dnp no)
 		(property "Reference" "#PWR011"
-			(at 90.17 68.58 0)
+			(at 90.17 66.04 0)
 			(effects
 				(font
@@
 		)
 		(property "Value" "+3V3"
-			(at 97.282 67.564 90)
+			(at 97.282 65.786 90)
 			(effects
 				(font
@@
 		)
 		(property "Footprint" ""
-			(at 93.98 68.58 0)
+			(at 93.98 66.04 0)
 			(effects
 				(font
@@
 		)
 		(property "Datasheet" ""
-			(at 93.98 68.58 0)
-			(effects
-				(font
-					(size 1.27 1.27)
-				)
-				(hide yes)
-			)
-		)
-		(property "Description" ""
-			(at 93.98 68.58 0)
-			(effects
-				(font
+			(at 93.98 66.04 0)
+			(effects
+				(font
+					(size 1.27 1.27)
+				)
+				(hide yes)
+			)
+		)
+		(property "Description" ""
+			(at 93.98 66.04 0)
+			(effects
+				(font
