File: elec/modules/buck/buck.kicad_sch (KiCad schematic)
At the start: 14 parts, among them J1 Conn_01x08, J2 Conn_01x08

Commit message: bucks done
Connections:
- net +3V3: now also C6.1, PS2.5 (SENSE)
- net +5V: now also C5.1, PS1.5 (SENSE)
- net at D1.2 (A), PS1.4 (VOUT): no longer C5.1, PS1.5 (SENSE)
- net at D2.2 (A), PS2.4 (VOUT): no longer C6.1, PS2.5 (SENSE)
Other:
- moved on the sheet: C5, C6, D1, D2
Changed lines of the file:
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@@
-	)
-	(junction
-		(at 162.56 62.23)
-		(diameter 0)
-		(color 0 0 0 0)
 	)
 	(junction
@@
 	)
 	(junction
-		(at 101.6 121.92)
+		(at 171.45 101.6)
 		(diameter 0)
 		(color 0 0 0 0)
 	)
 	(junction
-		(at 163.83 101.6)
+		(at 101.6 121.92)
 		(diameter 0)
 		(color 0 0 0 0)
@@
 	)
 	(junction
+		(at 166.37 62.23)
+		(diameter 0)
+		(color 0 0 0 0)
+	)
+	(junction
 		(at 71.12 59.69)
 		(diameter 0)
@@
 	)
 	(junction
-		(at 166.37 62.23)
+		(at 170.18 62.23)
 		(diameter 0)
 		(color 0 0 0 0)
@@
 	(wire
 		(pts
-			(xy 166.37 82.55) (xy 166.37 71.12)
+			(xy 170.18 82.55) (xy 170.18 81.28)
 		)
 		(stroke
@@
 	(wire
 		(pts
-			(xy 160.02 104.14) (xy 163.83 104.14)
+			(xy 160.02 104.14) (xy 167.64 104.14)
 		)
 		(stroke
@@
 	(wire
 		(pts
-			(xy 167.64 101.6) (xy 167.64 102.87)
+			(xy 171.45 101.6) (xy 171.45 102.87)
 		)
 		(stroke
@@
 	(wire
 		(pts
+			(xy 171.45 101.6) (xy 179.07 101.6)
+		)
+		(stroke
+			(width 0)
+			(type default)
+		)
+	)
+	(wire
+		(pts
 			(xy 71.12 82.55) (xy 81.28 82.55)
 		)
@@
 	(wire
 		(pts
+			(xy 166.37 64.77) (xy 166.37 62.23)
+		)
+		(stroke
+			(width 0)
+			(type default)
+		)
+	)
+	(wire
+		(pts
 			(xy 101.6 121.92) (xy 133.35 121.92)
 		)
@@
 	(wire
 		(pts
-			(xy 166.37 62.23) (xy 166.37 63.5)
+			(xy 170.18 62.23) (xy 170.18 73.66)
 		)
 		(stroke
@@
 	(wire
 		(pts
-			(xy 167.64 121.92) (xy 167.64 110.49)
+			(xy 171.45 121.92) (xy 171.45 110.49)
 		)
 		(stroke
@@
 	(wire
 		(pts
-			(xy 179.07 62.23) (xy 177.8 62.23)
-		)
-		(stroke
-			(width 0)
-			(type default)
-		)
-	)
-	(wire
-		(pts
 			(xy 81.28 59.69) (xy 102.87 59.69)
 		)
@@
 	(wire
 		(pts
-			(xy 158.75 62.23) (xy 162.56 62.23)
+			(xy 167.64 104.14) (xy 167.64 101.6)
+		)
+		(stroke
+			(width 0)
+			(type default)
+		)
+	)
+	(wire
+		(pts
+			(xy 166.37 62.23) (xy 170.18 62.23)
 		)
 		(stroke
@@
 	(wire
 		(pts
-			(xy 162.56 62.23) (xy 166.37 62.23)
-		)
-		(stroke
-			(width 0)
-			(type default)
-		)
-	)
-	(wire
-		(pts
-			(xy 132.08 82.55) (xy 166.37 82.55)
+			(xy 170.18 62.23) (xy 179.07 62.23)
+		)
+		(stroke
+			(width 0)
+			(type default)
+		)
+	)
+	(wire
+		(pts
+			(xy 132.08 82.55) (xy 170.18 82.55)
 		)
 		(stroke
@@
 	(wire
 		(pts
-			(xy 158.75 64.77) (xy 162.56 64.77)
-		)
-		(stroke
-			(width 0)
-			(type default)
-		)
-	)
-	(wire
-		(pts
-			(xy 179.07 101.6) (xy 177.8 101.6)
-		)
-		(stroke
-			(width 0)
-			(type default)
-		)
-	)
-	(wire
-		(pts
-			(xy 162.56 64.77) (xy 162.56 62.23)
+			(xy 158.75 64.77) (xy 166.37 64.77)
 		)
 		(stroke
@@
 	(wire
 		(pts
+			(xy 167.64 101.6) (xy 171.45 101.6)
+		)
+		(stroke
+			(width 0)
+			(type default)
+		)
+	)
+	(wire
+		(pts
 			(xy 72.39 114.3) (xy 72.39 121.92)
 		)
@@
 	(wire
 		(pts
-			(xy 133.35 121.92) (xy 167.64 121.92)
+			(xy 133.35 121.92) (xy 171.45 121.92)
 		)
 		(stroke
@@
 	(wire
 		(pts
-			(xy 170.18 101.6) (xy 167.64 101.6)
-		)
-		(stroke
-			(width 0)
-			(type default)
-		)
-	)
-	(wire
-		(pts
 			(xy 46.99 158.75) (xy 46.99 161.29)
 		)
@@
 	(wire
 		(pts
-			(xy 163.83 104.14) (xy 163.83 101.6)
-		)
-		(stroke
-			(width 0)
-			(type default)
-		)
-	)
-	(wire
-		(pts
 			(xy 81.28 82.55) (xy 91.44 82.55)
 		)
@@
 	(wire
 		(pts
-			(xy 163.83 101.6) (xy 167.64 101.6)
-		)
-		(stroke
-			(width 0)
-			(type default)
-		)
-	)
-	(wire
-		(pts
 			(xy 72.39 99.06) (xy 82.55 99.06)
 		)
@@
 	(wire
 		(pts
-			(xy 160.02 101.6) (xy 163.83 101.6)
-		)
-		(stroke
-			(width 0)
-			(type default)
-		)
-	)
-	(wire
-		(pts
 			(xy 104.14 104.14) (xy 101.6 104.14)
-		)
-		(stroke
-			(width 0)
-			(type default)
-		)
-	)
-	(wire
-		(pts
-			(xy 170.18 62.23) (xy 166.37 62.23)
 		)
 		(stroke
@@
 	(symbol
 		(lib_id "Device:C_Polarized")
-		(at 166.37 67.31 0)
+		(at 170.18 77.47 0)
 		(unit 1)
 		(exclude_from_sim no)
@@
 		(dnp no)
 		(property "Reference" "C5"
-			(at 170.18 65.1509 0)
+			(at 173.99 75.3109 0)
 			(effects
 				(font
@@
 		)
 		(property "Value" "220u"
-			(at 170.18 67.6909 0)
+			(at 173.99 77.8509 0)
 			(effects
 				(font
@@
 		)
 		(property "Footprint" "Capacitor_Tantalum_SMD:CP_EIA-7343-15_Kemet-W_HandSolder"
-			(at 167.3352 71.12 0)
+			(at 171.1452 81.28 0)
 			(effects
 				(font
@@
 		)
 		(property "Datasheet" "~"
-			(at 166.37 67.31 0)
+			(at 170.18 77.47 0)
 			(effects
 				(font
@@
 		)
 		(property "Description" ""
-			(at 166.37 67.31 0)
+			(at 170.18 77.47 0)
 			(effects
 				(font
@@
 	(symbol
 		(lib_id "Diode:B340")
-		(at 173.99 62.23 180)
+		(at 162.56 62.23 180)
 		(unit 1)
 		(exclude_from_sim no)
@@
 		(fields_autoplaced yes)
 		(property "Reference" "D1"
-			(at 174.3075 55.88 0)
+			(at 162.8775 55.88 0)
 			(effects
 				(font
@@
 		)
 		(property "Value" "SS54"
-			(at 174.3075 58.42 0)
+			(at 162.8775 58.42 0)
 			(effects
 				(font
@@
 		)
 		(property "Footprint" "Buck:DIOM5025X220N"
-			(at 173.99 57.785 0)
+			(at 162.56 57.785 0)
 			(effects
 				(font
@@
 		)
 		(property "Datasheet" "http://www.jameco.com/Jameco/Products/ProdDS/1538777.pdf"
-			(at 173.99 62.23 0)
+			(at 162.56 62.23 0)
 			(effects
 				(font
@@
 		)
 		(property "Description" ""
-			(at 173.99 62.23 0)
+			(at 162.56 62.23 0)
 			(effects
 				(font
@@
 	(symbol
 		(lib_id "Diode:B340")
-		(at 173.99 101.6 180)
-		(unit 1)
-		(exclude_from_sim no)
-		(in_bom yes)
-		(on_board yes)
-		(dnp no)
-		(fields_autoplaced yes)
+		(at 163.83 101.6 180)
+		(unit 1)
+		(exclude_from_sim no)
+		(in_bom yes)
+		(on_board yes)
+		(dnp no)
 		(property "Reference" "D2"
-			(at 174.3075 95.25 0)
+			(at 164.1475 95.25 0)
 			(effects
 				(font
@@
 		)
 		(property "Value" "SS54"
-			(at 174.3075 97.79 0)
+			(at 164.1475 97.79 0)
 			(effects
 				(font
@@
 		)
 		(property "Footprint" "Buck:DIOM5025X220N"
-			(at 173.99 97.155 0)
+			(at 163.83 97.155 0)
 			(effects
 				(font
@@
 		)
 		(property "Datasheet" "http://www.jameco.com/Jameco/Products/ProdDS/1538777.pdf"
-			(at 173.99 101.6 0)
+			(at 163.83 101.6 0)
 			(effects
 				(font
@@
 		)
 		(property "Description" ""
-			(at 173.99 101.6 0)
+			(at 163.83 101.6 0)
 			(effects
 				(font
@@
 	(symbol
 		(lib_id "Device:C_Polarized")
-		(at 167.64 106.68 0)
+		(at 171.45 106.68 0)
 		(unit 1)
 		(exclude_from_sim no)
@@
 		(dnp no)
 		(property "Reference" "C6"
-			(at 171.45 104.5209 0)
+			(at 175.26 104.5209 0)
 			(effects
 				(font
@@
 		)
 		(property "Value" "220u"
-			(at 171.45 107.0609 0)
+			(at 175.26 107.0609 0)
 			(effects
 				(font
@@
 		)
 		(property "Footprint" "Capacitor_Tantalum_SMD:CP_EIA-7343-15_Kemet-W_HandSolder"
-			(at 168.6052 110.49 0)
+			(at 172.4152 110.49 0)
 			(effects
 				(font
@@
 		)
 		(property "Datasheet" "~"
-			(at 167.64 106.68 0)
+			(at 171.45 106.68 0)
 			(effects
 				(font
@@
 		)
 		(property "Description" ""
-			(at 167.64 106.68 0)
-			(effects
-				(font
+			(at 171.45 106.68 0)
+			(effects
+				(font
