File: elec/modules/solactivation/solactivation.kicad_pcb (KiCad board)
At the start: 2 copper layers, 30.5 x 40.6 mm, 11 parts, among them J1 Conn_01x08, J2 Conn_01x08, J5 XT30, Q1 STP75NF75, Q2 IRLML6344TRPBF

Commit message: added name cos why not
Other:
- board text added: "Design By Euston Tan"
Changed lines of the file:
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@@
 		(layer "Edge.Cuts")
+	)
+	(gr_text "Design By Euston Tan \n"
+		(at 144.74 117.28 0)
+		(layer "B.SilkS")
+		(effects
+			(font
+				(size 1 1)
+				(thickness 0.2)
+				(bold yes)
+			)
+			(justify mirror)
+		)
 	)
 	(gr_text "design of 2-Chairs. 2025\nJLC Order No. JLCJLCJLCJLC"

Commit message: chore: production files; chore: rev num for solactivation
Routing:
- added copper zone on B.Cu, net Net-(D37-A)
Other:
- board text added: "design of 2-Chairs. 2025 JLC Order No. JLCJLCJLCJLC rev 1.0"
- board text removed: "design of 2-Chairs. 2025 JLC Order No. JLCJLCJLCJLC"
Changed lines of the file:
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@@
 	)
 	(paper "A4")
+	(title_block
+		(title "Solenoid Activation")
+		(date "2025-12-02")
+		(rev "1.0")
+		(company "2-Chairs. 2025")
+	)
 	(layers
 		(0 "F.Cu" signal)
@@
 		)
 	)
-	(gr_text "design of 2-Chairs. 2025\nJLC Order No. JLCJLCJLCJLC"
-		(at 144.24 89.03 0)
+	(gr_text "design of 2-Chairs. 2025\nJLC Order No. JLCJLCJLCJLC\nrev 1.0"
+		(at 144.74 90.03 0)
 		(layer "B.SilkS")
 		(effects
@@
 	)
 	(zone
-		(net 1)
-		(net_name "Net-(C4-Pad1)")
+		(net 5)
+		(net_name "/Sol")
 		(layer "F.Cu")
-		(hatch edge 0.5)
-		(priority 3)
+		(name "$teardrop_padvia$")
+		(hatch none 0.1)
+		(priority 30001)
+		(attr
+			(teardrop
+				(type padvia)
+			)
+		)
 		(connect_pads yes
-			(clearance 0.5)
+			(clearance 0)
 		)
-		(min_thickness 0.25)
+		(min_thickness 0.0254)
 		(filled_areas_thickness no)
 		(fill yes
 			(thermal_gap 0.5)
 			(thermal_bridge_width 0.5)
-			(smoothing chamfer)
-			(radius 0.25)
+			(island_removal_mode 1)
+			(island_area_min 10)
 		)
 		(polygon
 			(pts
-				(xy 150.49 96.73) (xy 150.49 100.78) (xy 148.49 100.78) (xy 148.49 96.73)
+				(xy 149.44 91.68) (xy 149.44 92.28) (xy 149.97956 92.507574) (xy 150.441 92.03) (xy 150.001732 91.537612)
 			)
 		)
 	)
 	(zone
-		(net 3)
-		(net_name "Net-(D37-A)")
+		(net 5)
+		(net_name "/Sol")
 		(layer "F.Cu")
-		(hatch edge 0.5)
-		(priority 4)
+		(name "$teardrop_padvia$")
+		(hatch none 0.1)
+		(priority 30000)
+		(attr
+			(teardrop
+				(type padvia)
+			)
+		)
 		(connect_pads yes
-			(clearance 0.5)
+			(clearance 0)
 		)
-		(min_thickness 0.25)
+		(min_thickness 0.0254)
 		(filled_areas_thickness no)
 		(fill yes
 			(thermal_gap 0.5)
 			(thermal_bridge_width 0.5)
-			(smoothing chamfer)
-			(radius 0.25)
+			(island_removal_mode 1)
+			(island_area_min 10)
 		)
 		(polygon
 			(pts
-				(xy 144.75 113.28) (xy 144.75 116.03) (xy 154.49 116.03) (xy 154.49 100.78) (xy 148.49 100.78) (xy 148.49 97.28)
-				(xy 142.24 97.28) (xy 142.24 99.78) (xy 146.99 99.78) (xy 146.99 103.53) (xy 144.74 103.53) (xy 144.74 113.27)
+				(xy 149.449607 91.68) (xy 149.449607 92.28) (xy 150.342455 92.520393) (xy 150.441 92.03) (xy 150.342455 91.539607)
 			)
 		)
 	)
 	(zone
-		(net 4)
-		(net_name "+24V")
+		(net 1)
+		(net_name "Net-(C4-Pad1)")
 		(layer "F.Cu")
 		(hatch edge 0.5)
-		(priority 1)
+		(priority 3)
 		(connect_pads yes
 			(clearance 0.5)
@@
 		(polygon
 			(pts
-				(xy 144.75 104.28) (xy 133.49 104.28) (xy 133.49 122.03) (xy 144.75 122.03)
+				(xy 150.49 96.73) (xy 150.49 100.78) (xy 148.49 100.78) (xy 148.49 96.73)
 			)
 		)
 	)
 	(zone
-		(net 7)
-		(net_name "+12V")
+		(net 3)
+		(net_name "Net-(D37-A)")
 		(layer "F.Cu")
 		(hatch edge 0.5)
-		(priority 6)
+		(priority 4)
 		(connect_pads yes
 			(clearance 0.5)
@@
 		(polygon
 			(pts
-				(xy 142.24 100.78) (xy 133.99 100.78) (xy 133.99 83.53) (xy 142.24 83.53) (xy 142.24 90.28) (xy 138.74 90.28)
-				(xy 138.74 96.73) (xy 142.24 96.73)
+				(xy 144.75 113.28) (xy 144.75 115.03) (xy 154.49 115.03) (xy 154.49 100.78) (xy 148.49 100.78) (xy 148.49 97.28)
+				(xy 144.24 97.28) (xy 144.24 99.78) (xy 146.99 99.78) (xy 146.99 103.53) (xy 144.74 103.53) (xy 144.74 113.27)
 			)
 		)
 	)
 	(zone
-		(net 5)
-		(net_name "/Sol")
+		(net 4)
+		(net_name "+24V")
 		(layer "F.Cu")
-		(name "$teardrop_padvia$")
-		(hatch none 0.1)
-		(priority 30000)
-		(attr
-			(teardrop
-				(type padvia)
-			)
-		)
+		(hatch edge 0.5)
+		(priority 1)
 		(connect_pads yes
-			(clearance 0)
+			(clearance 0.5)
 		)
-		(min_thickness 0.0254)
+		(min_thickness 0.25)
 		(filled_areas_thickness no)
 		(fill yes
 			(thermal_gap 0.5)
 			(thermal_bridge_width 0.5)
-			(island_removal_mode 1)
-			(island_area_min 10)
+			(smoothing chamfer)
+			(radius 0.25)
 		)
 		(polygon
 			(pts
-				(xy 149.449607 91.68) (xy 149.449607 92.28) (xy 150.342455 92.520393) (xy 150.441 92.03) (xy 150.342455 91.539607)
+				(xy 144.75 104.28) (xy 133.49 104.28) (xy 133.49 122.03) (xy 144.75 122.03)
 			)
 		)
 	)
 	(zone
-		(net 5)
-		(net_name "/Sol")
+		(net 7)
+		(net_name "+12V")
 		(layer "F.Cu")
-		(name "$teardrop_padvia$")
-		(hatch none 0.1)
-		(priority 30001)
-		(attr
-			(teardrop
-				(type padvia)
-			)
-		)
+		(hatch edge 0.5)
+		(priority 6)
 		(connect_pads yes
-			(clearance 0)
+			(clearance 0.5)
 		)
-		(min_thickness 0.0254)
+		(min_thickness 0.25)
 		(filled_areas_thickness no)
 		(fill yes
 			(thermal_gap 0.5)
 			(thermal_bridge_width 0.5)
-			(island_removal_mode 1)
-			(island_area_min 10)
+			(smoothing chamfer)
+			(radius 0.25)
 		)
 		(polygon
 			(pts
-				(xy 149.44 91.68) (xy 149.44 92.28) (xy 149.97956 92.507574) (xy 150.441 92.03) (xy 150.001732 91.537612)
+				(xy 144.09 100.78) (xy 133.99 100.78) (xy 133.99 83.53) (xy 142.24 83.53) (xy 142.24 90.28) (xy 138.74 90.28)
+				(xy 138.74 96.73) (xy 144.09 96.73)
 			)
 		)
@@
 	)
 	(zone
+		(net 3)
+		(net_name "Net-(D37-A)")
+		(layer "B.Cu")
+		(hatch edge 0.5)
+		(priority 7)
+		(connect_pads yes
+			(clearance 0.5)
+		)
+		(min_thickness 0.25)
+		(filled_areas_thickness no)
+		(fill yes
+			(thermal_gap 0.5)
+			(thermal_bridge_width 0.5)
+			(smoothing chamfer)
+			(radius 0.25)
+		)
+		(polygon
+			(pts
+				(xy 154.49 115.03) (xy 144.7492 115.03) (xy 144.739 102.28) (xy 146.99 102.28) (xy 146.99 99.78)
+				(xy 144.24 99.78) (xy 144.24 97.28) (xy 154.49 97.28)
+			)
+		)
+	)
+	(zone
 		(net 5)
 		(net_name "/Sol")
@@
 		(name "$teardrop_padvia$")
 		(hatch none 0.1)
-		(priority 30000)
+		(priority 30003)
 		(attr
 			(teardrop
@@
 		(polygon
 			(pts
-				(xy 145.725 86.968667) (xy 146.325 86.968667) (xy 146.858667 85.450827) (xy 146.025 85.284) (xy 145.191333 85.450827)
+				(xy 149.449607 91.73) (xy 149.449607 92.33) (xy 150.342455 92.520393) (xy 150.441 92.03) (xy 150.342455 91.539607)
 			)
 		)
@@
 		(name "$teardrop_padvia$")
 		(hatch none 0.1)
-		(priority 30001)
+		(priority 30002)
 		(attr
 			(teardrop
@@
 		(polygon
 			(pts
-				(xy 144.341333 84.985) (xy 144.341333 85.585) (xy 145.859173 86.118667) (xy 146.026 85.285) (xy 145.859173 84.451333)
+				(xy 145.725 86.968667) (xy 146.325 86.968667) (xy 146.858667 85.450827) (xy 146.025 85.284) (xy 145.191333 85.450827)
 			)
 		)
@@
 		(name "$teardrop_padvia$")
 		(hatch none 0.1)
-		(priority 30002)
+		(priority 30000)
 		(attr
 			(teardrop
@@
 		(polygon
 			(pts
-				(xy 145.168667 85.585) (xy 145.168667 84.985) (xy 143.650827 84.451333) (xy 143.484 85.285) (xy 143.650827 86.118667)
+				(xy 144.341333 84.985) (xy 144.341333 85.585) (xy 145.859173 86.118667) (xy 146.026 85.285) (xy 145.859173 84.451333)
 			)
 		)
@@
 		(name "$teardrop_padvia$")
 		(hatch none 0.1)
-		(priority 30003)
+		(priority 30001)
 		(attr
 			(teardrop
@@
 		(polygon
 			(pts
-				(xy 149.449607 91.73) (xy 149.449607 92.33) (xy 150.342455 92.520393) (xy 150.441 92.03) (xy 150.342455 91.539607)
+				(xy 145.168667 85.585) (xy 145.168667 84.985) (xy 143.650827 84.451333) (xy 143.484 85.285) (xy 143.650827 86.118667)
 			)
 		)
