File: elec/modules/solactivation/solactivation.kicad_sch (KiCad schematic)
At the start: 12 parts, among them J1 Conn_01x01_Pin, J3 Conn_01x01_Pin, J4 Conn_01x01_Pin, J5 XT30, Q1 STP75NF75, Q2 IRLML6344TRPBF

Commit message: did stuff
Parts:
- removed J1, J3, J4: Conn_01x01_Pin, cool custom thingy:custompadfat, symbol Connector:Conn_01x01_Pin
- added J1, J2: Conn_01x08, symbol Connector_Generic:Conn_01x08
Connections:
- net +12V: now also J1.1 (Pin_1), J1.2 (Pin_2), J1.3 (Pin_3)
- net +24V: now also J2.1 (Pin_1), J2.2 (Pin_2), J2.3 (Pin_3), J2.4 (Pin_4)
- net GND: now also J1.6 (Pin_6), J1.7 (Pin_7), J1.8 (Pin_8), J2.6 (Pin_6), J2.7 (Pin_7), J2.8 (Pin_8)
- net Sol: now also J1.4 (Pin_4), J1.5 (Pin_5)
- no-connect marks 0 -> 1

Commit message: finished pcbs-silkscrfeen pcbs seem halal
Parts:
- J1, J2: footprint (none) -> Connector_PinSocket_2.54mm:PinSocket_1x08_P2.54mm_Vertical
Changed lines of the file:
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@@
 			)
 		)
-		(property "Footprint" ""
+		(property "Footprint" "Connector_PinSocket_2.54mm:PinSocket_1x08_P2.54mm_Vertical"
 			(at 186.69 129.54 0)
 			(effects
@@
 			)
 		)
-		(property "Footprint" ""
+		(property "Footprint" "Connector_PinSocket_2.54mm:PinSocket_1x08_P2.54mm_Vertical"
 			(at 149.86 129.54 0)
 			(effects

Commit message: chore: production files; chore: rev num for solactivation
Other:
- company: (none) -> 2-Chairs. 2025
- title: (none) -> Solenoid Activation
Changed lines of the file:
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@@
 	(generator_version "9.0")
 	(paper "A4")
+	(title_block
+		(title "Solenoid Activation")
+		(date "2025-12-02")
+		(rev "1.0")
+		(company "2-Chairs. 2025")
+	)
 	(junction
 		(at 120.65 66.04)

Commit message: stuff
Other:
- moved on the sheet: J1
Changed lines of the file:
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@@
 	(wire
 		(pts
-			(xy 144.78 137.16) (xy 144.78 134.62)
-		)
-		(stroke
-			(width 0)
-			(type default)
-		)
-	)
-	(wire
-		(pts
-			(xy 161.29 137.16) (xy 157.48 137.16)
+			(xy 181.61 119.38) (xy 181.61 116.84)
+		)
+		(stroke
+			(width 0)
+			(type default)
+		)
+	)
+	(wire
+		(pts
+			(xy 198.12 119.38) (xy 194.31 119.38)
 		)
 		(stroke
@@
 	(wire
 		(pts
-			(xy 147.32 139.7) (xy 137.16 139.7)
+			(xy 184.15 121.92) (xy 173.99 121.92)
 		)
 		(stroke
@@
 	(wire
 		(pts
-			(xy 139.7 137.16) (xy 144.78 137.16)
+			(xy 176.53 119.38) (xy 181.61 119.38)
 		)
 		(stroke
@@
 	(wire
 		(pts
-			(xy 147.32 134.62) (xy 147.32 139.7)
+			(xy 184.15 116.84) (xy 184.15 121.92)
 		)
 		(stroke
@@
 	(wire
 		(pts
-			(xy 157.48 137.16) (xy 157.48 134.62)
+			(xy 194.31 119.38) (xy 194.31 116.84)
 		)
 		(stroke
@@
 	(wire
 		(pts
-			(xy 162.56 139.7) (xy 154.94 139.7)
+			(xy 199.39 121.92) (xy 191.77 121.92)
 		)
 		(stroke
@@
 	(wire
 		(pts
-			(xy 154.94 139.7) (xy 154.94 134.62)
+			(xy 191.77 121.92) (xy 191.77 116.84)
 		)
 		(stroke
@@
 	)
 	(label "Sol"
-		(at 149.86 134.62 270)
+		(at 186.69 116.84 270)
 		(effects
 			(font
@@
 	)
 	(label "Sol"
-		(at 152.4 134.62 270)
+		(at 189.23 116.84 270)
 		(effects
 			(font
@@
 	(symbol
 		(lib_id "power:GND")
-		(at 161.29 137.16 90)
+		(at 198.12 119.38 90)
 		(unit 1)
 		(exclude_from_sim no)
@@
 		(fields_autoplaced yes)
 		(property "Reference" "#PWR04"
-			(at 167.64 137.16 0)
+			(at 204.47 119.38 0)
 			(effects
 				(font
@@
 		)
 		(property "Value" "GND"
-			(at 165.1 137.1599 90)
+			(at 201.93 119.3799 90)
 			(effects
 				(font
@@
 		)
 		(property "Footprint" ""
-			(at 161.29 137.16 0)
+			(at 198.12 119.38 0)
 			(effects
 				(font
@@
 		)
 		(property "Datasheet" ""
-			(at 161.29 137.16 0)
+			(at 198.12 119.38 0)
 			(effects
 				(font
@@
 		)
 		(property "Description" ""
-			(at 161.29 137.16 0)
+			(at 198.12 119.38 0)
 			(effects
 				(font
@@
 	(symbol
 		(lib_id "power:+12V")
-		(at 139.7 137.16 90)
+		(at 176.53 119.38 90)
 		(unit 1)
 		(exclude_from_sim no)
@@
 		(dnp no)
 		(property "Reference" "#PWR03"
-			(at 143.51 137.16 0)
+			(at 180.34 119.38 0)
 			(effects
 				(font
@@
 		)
 		(property "Value" "+12V"
-			(at 131.572 136.144 90)
+			(at 168.402 118.364 90)
 			(effects
 				(font
@@
 		)
 		(property "Footprint" ""
-			(at 139.7 137.16 0)
+			(at 176.53 119.38 0)
 			(effects
 				(font
@@
 		)
 		(property "Datasheet" ""
-			(at 139.7 137.16 0)
+			(at 176.53 119.38 0)
 			(effects
 				(font
@@
 		)
 		(property "Description" ""
-			(at 139.7 137.16 0)
+			(at 176.53 119.38 0)
 			(effects
 				(font
@@
 	(symbol
 		(lib_id "power:GND")
-		(at 160.02 134.62 90)
+		(at 196.85 116.84 90)
 		(unit 1)
 		(exclude_from_sim no)
@@
 		(fields_autoplaced yes)
 		(property "Reference" "#PWR036"
-			(at 166.37 134.62 0)
+			(at 203.2 116.84 0)
 			(effects
 				(font
@@
 		)
 		(property "Value" "GND"
-			(at 163.83 134.6199 90)
+			(at 200.66 116.8399 90)
 			(effects
 				(font
@@
 		)
 		(property "Footprint" ""
-			(at 160.02 134.62 0)
+			(at 196.85 116.84 0)
 			(effects
 				(font
@@
 		)
 		(property "Datasheet" ""
-			(at 160.02 134.62 0)
+			(at 196.85 116.84 0)
 			(effects
 				(font
@@
 		)
 		(property "Description" ""
-			(at 160.02 134.62 0)
+			(at 196.85 116.84 0)
 			(effects
 				(font
@@
 	(symbol
 		(lib_id "power:+12V")
-		(at 137.16 139.7 90)
+		(at 173.99 121.92 90)
 		(unit 1)
 		(exclude_from_sim no)
@@
 		(dnp no)
 		(property "Reference" "#PWR05"
-			(at 140.97 139.7 0)
+			(at 177.8 121.92 0)
 			(effects
 				(font
@@
 		)
 		(property "Value" "+12V"
-			(at 129.032 138.684 90)
+			(at 165.862 120.904 90)
 			(effects
 				(font
@@
 		)
 		(property "Footprint" ""
-			(at 137.16 139.7 0)
+			(at 173.99 121.92 0)
 			(effects
 				(font
@@
 		)
 		(property "Datasheet" ""
-			(at 137.16 139.7 0)
+			(at 173.99 121.92 0)
 			(effects
 				(font
@@
 		)
 		(property "Description" ""
-			(at 137.16 139.7 0)
+			(at 173.99 121.92 0)
 			(effects
 				(font
@@
 	(symbol
 		(lib_id "power:GND")
-		(at 162.56 139.7 90)
+		(at 199.39 121.92 90)
 		(unit 1)
 		(exclude_from_sim no)
@@
 		(fields_autoplaced yes)
 		(property "Reference" "#PWR06"
-			(at 168.91 139.7 0)
+			(at 205.74 121.92 0)
 			(effects
 				(font
@@
 		)
 		(property "Value" "GND"
-			(at 166.37 139.6999 90)
+			(at 203.2 121.9199 90)
 			(effects
 				(font
@@
 		)
 		(property "Footprint" ""
-			(at 162.56 139.7 0)
+			(at 199.39 121.92 0)
 			(effects
 				(font
@@
 		)
 		(property "Datasheet" ""
-			(at 162.56 139.7 0)
+			(at 199.39 121.92 0)
 			(effects
 				(font
@@
 		)
 		(property "Description" ""
-			(at 162.56 139.7 0)
+			(at 199.39 121.92 0)
 			(effects
 				(font
@@
 	(symbol
 		(lib_id "Connector_Generic:Conn_01x08")
-		(at 149.86 129.54 90)
+		(at 186.69 111.76 90)
 		(unit 1)
 		(exclude_from_sim no)
@@
 		(fields_autoplaced yes)
 		(property "Reference" "J1"
-			(at 151.13 123.19 90)
+			(at 187.96 105.41 90)
 			(effects
 				(font
@@
 		)
 		(property "Value" "Conn_01x08"
-			(at 151.13 125.73 90)
+			(at 187.96 107.95 90)
 			(effects
 				(font
@@
 		)
 		(property "Footprint" "Connector_PinSocket_2.54mm:PinSocket_1x08_P2.54mm_Vertical"
-			(at 149.86 129.54 0)
+			(at 186.69 111.76 0)
 			(effects
 				(font
@@
 		)
 		(property "Datasheet" "~"
-			(at 149.86 129.54 0)
+			(at 186.69 111.76 0)
 			(effects
 				(font
@@
 		)
 		(property "Description" "Generic connector, single row, 01x08, script generated (kicad-library-utils/schlib/autogen/connector/)"
-			(at 149.86 129.54 0)
+			(at 186.69 111.76 0)
 			(effects
 				(font
@@
 	(symbol
 		(lib_id "power:+12V")
-		(at 142.24 134.62 90)
+		(at 179.07 116.84 90)
 		(unit 1)
 		(exclude_from_sim no)
@@
 		(dnp no)
 		(property "Reference" "#PWR033"
-			(at 146.05 134.62 0)
+			(at 182.88 116.84 0)
 			(effects
 				(font
@@
 		)
 		(property "Value" "+12V"
-			(at 134.112 133.604 90)
+			(at 170.942 115.824 90)
 			(effects
 				(font
@@
 		)
 		(property "Footprint" ""
-			(at 142.24 134.62 0)
+			(at 179.07 116.84 0)
 			(effects
 				(font
@@
 		)
 		(property "Datasheet" ""
-			(at 142.24 134.62 0)
+			(at 179.07 116.84 0)
 			(effects
 				(font
@@
 		)
 		(property "Description" ""
-			(at 142.24 134.62 0)
-			(effects
-				(font
+			(at 179.07 116.84 0)
+			(effects
+				(font
