File: elec/modules/boost/boost.kicad_pcb (KiCad board)
At the start: 2 copper layers, 30.5 x 40.6 mm, 12 parts, among them J1 Conn_01x08, J2 Conn_01x08, U1 LM2587S-ADJ

Commit message: added name cos why not
Other:
- board text added: "Design By Euston Tan"
Changed lines of the file:
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@@
 		(layer "Edge.Cuts")
+	)
+	(gr_text "Design By Euston Tan \n"
+		(at 138.71 119.119999 0)
+		(layer "B.SilkS")
+		(effects
+			(font
+				(size 1 1)
+				(thickness 0.2)
+				(bold yes)
+			)
+			(justify mirror)
+		)
 	)
 	(gr_text "design of 2-Chairs. 2025\nJLC Order No. JLCJLCJLCJLC"

Commit message: chore: boost production files
Other:
- board text added: "design of 2-Chairs. 2025 JLC Order No. JLCJLCJLCJLC rev. 1.0"
- board text removed: "design of 2-Chairs. 2025 JLC Order No. JLCJLCJLCJLC"
Changed lines of the file:
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@@
 		(sheetname "/")
 		(sheetfile "boost.kicad_sch")
-		(attr through_hole exclude_from_pos_files)
+		(attr through_hole exclude_from_pos_files exclude_from_bom)
 		(fp_line
 			(start -1.33 -1.33)
@@
 		(sheetname "/")
 		(sheetfile "boost.kicad_sch")
-		(attr through_hole)
+		(attr through_hole exclude_from_pos_files exclude_from_bom)
 		(fp_line
 			(start -2.659698 -2.315)
@@
 		(sheetname "/")
 		(sheetfile "boost.kicad_sch")
-		(attr through_hole exclude_from_pos_files)
+		(attr through_hole exclude_from_pos_files exclude_from_bom)
 		(fp_line
 			(start -2.57 -3.26)
@@
 		(sheetname "/")
 		(sheetfile "boost.kicad_sch")
-		(attr through_hole exclude_from_pos_files)
+		(attr through_hole exclude_from_pos_files exclude_from_bom)
 		(fp_line
 			(start -1.33 -1.33)
@@
 		(sheetname "/")
 		(sheetfile "boost.kicad_sch")
-		(attr through_hole exclude_from_pos_files)
+		(attr through_hole exclude_from_pos_files exclude_from_bom)
 		(fp_line
 			(start -2.659698 -2.315)
@@
 		)
 	)
-	(gr_text "design of 2-Chairs. 2025\nJLC Order No. JLCJLCJLCJLC"
-		(at 138.71 111.119999 0)
+	(gr_text "design of 2-Chairs. 2025\nJLC Order No. JLCJLCJLCJLC\nrev. 1.0"
+		(at 138.71 110.119999 0)
 		(layer "B.SilkS")
 		(effects
