File: elec/modules/Tofs/XM125_Breakout.kicad_sch (KiCad schematic)
At the start: 46 parts, among them J1 USB_C_2-LAYER_PADS, J13 SWD (DNP), J14 CONN_09NO_SILK, J15 CONN_111X11_NO_SILK, J2 RIGHT_ANGLE, J3 RIGHT_ANGLE, U1 XM125, U2 RT9080-33GJ5, U3 RT9080-18GJ5, U4 CH340C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

Commit message: made schematics more organised ish for tofs
Hope i didnt mess anyuthingn  up
Parts:
- removed unit 2 of FRAME2
- removed LOGO1: SPECIAL_INSTRUCTIONS-ORDERING, XM125_Breakout:ORDERING_INSTRUCTIONS, symbol XM125_Breakout-eagle-import:SPECIAL_INSTRUCTIONS-ORDERING
- removed LOGO2: QWIIC_LOGO_4MM, XM125_Breakout:QWIIC_4MM, symbol XM125_Breakout-eagle-import:QWIIC_LOGO_4MM
- removed LOGO3, LOGO6: SFE_LOGO_NAME_FLAME.1_INCH, XM125_Breakout:SFE_LOGO_NAME_FLAME_.1, symbol XM125_Breakout-eagle-import:SFE_LOGO_NAME_FLAME.1_INCH
- removed LOGO4: OSHW-LOGOS, XM125_Breakout:OSHW-LOGO-S, symbol XM125_Breakout-eagle-import:OSHW-LOGOS
- removed LOGO5: SFE_LOGO_FLAME.1_INCH, XM125_Breakout:SFE_LOGO_FLAME_.1, symbol XM125_Breakout-eagle-import:SFE_LOGO_FLAME.1_INCH
Other:
- moved on the sheet: C1, S1, S2
