File: elec/modules/Lightfgate(LDR)/Lightfgate(LDR).kicad_pcb (KiCad board)
At the start: 2 copper layers, 24.4 x 47.7 mm, 2 parts, among them J1 Conn_01x02

Commit message: idk
Parts:
- J1: footprint Pinheaders:PinHeader_1x02_P2.54mm_Vertical -> Connector_JST:JST_SH_BM02B-SRSS-TB_1x02-1MP_P1.00mm_Vertical
- moved J1 57.2 mm to (162.8, 114.7)
- moved LED_2 38.3 mm to (151.0, 103.6), turned to 90 degrees
Routing:
- added copper zone on B.Cu, net +3V3
- added copper zone on F.Cu, net +3V3
