File: elec/modules/Lightgate(LED)/Lightgate(LED).kicad_sch (KiCad schematic)
At the start: 2 parts, among them J1 Conn_01x02

Commit message: idk
Parts:
- J1: footprint Pinheaders:PinHeader_1x02_P2.54mm_Vertical -> Connector_JST:JST_SH_BM02B-SRSS-TB_1x02-1MP_P1.00mm_Vertical
Changed lines of the file:
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@@
 			)
 		)
-		(property "Footprint" "Pinheaders:PinHeader_1x02_P2.54mm_Vertical"
+		(property "Footprint" "Connector_JST:JST_SH_BM02B-SRSS-TB_1x02-1MP_P1.00mm_Vertical"
 			(at 120.65 100.33 0)
 			(effects
