File: elec/layer1/layer1.kicad_pcb (KiCad board)
At the start: 2 copper layers, 178 x 173.3 mm, 114 parts, among them U1 DEV-15583, U2 CD74HC4067SM, U3 CD74HC4067SM

Commit message: Revert "driver jsts r almost done ig"
This reverts commit 0dd8e7197cd13faec0b768cbe0f6c1db0f8b679d.
Parts:
- removed Driver5, Driver6, Driver7, Driver8: Conn_01x08, Pinheaders:PinHeader_1x08_P2.54mm_Vertical
- added L1-->L2Connection1: Conn_01x08, L1:PinHeader_1x08_P2.54mm_Vertical, F.Cu at (219.8, 73.1)
- moved L1-->L2Connection2 12.1 mm to (176.7, 73.1)
- moved Driver2 1.40 mm to (260.1, 170.2)
- moved Driver1 1.40 mm to (260.1, 135.5)
Connections:
- L1-->L2Connection2 pad 1: +5V -> +12V
- L1-->L2Connection2 pad 2: +5V -> +12V
- L1-->L2Connection2 pad 3: unconnected-(L1--&gt;L2Connection2-Pin_3-Pad3) -> +12V
- U1 pad 0: unconnected-(U1-Pad0) -> /M2 IN B
- U1 pad 10: unconnected-(U1-Pad10) -> /M2 PWM
- U1 pad 19: unconnected-(U1-Pad19) -> /Mux Com (1-16)
- U1 pad 20: unconnected-(U1-Pad20) -> /Sol
- U1 pad 21: unconnected-(U1-Pad21) -> /M2 IN A
- U1 pad 22: unconnected-(U1-Pad22) -> /M1 IN A
- U1 pad 23: unconnected-(U1-Pad23) -> /M1 IN B
- U1 pad 9: unconnected-(U1-Pad9) -> /M1 PWM
Routing:
- net /M SW: track 4.99 -> 248.3 mm, vias 0 -> 2
- net +12V: track 30.5 -> 254.4 mm, vias 0 -> 1
- net /M2 IN B: track 4.99 -> 128.7 mm, vias 0 -> 1
- net /M1 PWM: track 0.00 -> 120.9 mm
- net /M1 IN A: track 0.00 -> 120.4 mm
- net /M2 PWM: track 4.99 -> 123.7 mm
- net /M2 IN A: track 4.99 -> 109.4 mm, vias 0 -> 1
- net /M1 IN B: track 0.00 -> 101.1 mm
- net +3V3: track 130.3 -> 178.4 mm
- net unconnected-(U1-Pad21): track 21.5 -> 0.00 mm
- net +5V: track 53.4 -> 36.4 mm
- net /RX: track 6.29 -> 11.3 mm
- net /TX: track 6.29 -> 11.0 mm
- net unconnected-(U1-Pad9): track 3.74 -> 0.00 mm
- net unconnected-(U1-Pad22): track 1.23 -> 0.00 mm
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Other:
- board text added: "12v"
- board text added: "5v"
- board text added: "Gnd"
- board text added: "Rx"
- board text added: "Tx"

Commit message: l2 domne
Parts:
- added Driver5: Conn_01x08, Pinheaders:PinHeader_1x08_P2.54mm_Vertical, F.Cu at (119.9, 130.2)
- added Driver6: Conn_01x08, Pinheaders:PinHeader_1x08_P2.54mm_Vertical, F.Cu at (42.5, 108.2)
- added Driver7: Conn_01x08, Pinheaders:PinHeader_1x08_P2.54mm_Vertical, F.Cu at (47.2, 108.2)
- added Driver8: Conn_01x08, Pinheaders:PinHeader_1x08_P2.54mm_Vertical, F.Cu at (51.8, 108.2)
- L1-->l2Connection1: renamed from L1-->L2Connection1; value Conn_01x08 -> Conn_01x09; footprint L1:PinHeader_1x08_P2.54mm_Vertical -> Pinheaders:PinHeader_1x09_P2.54mm_Vertical
Connections:
- L1-->l2Connection1 pad 1: +3V3 -> /Dribbler Data
- L1-->l2Connection1 pad 2: +3V3 -> /LightGateLDR
- L1-->l2Connection1 pad 3: +3V3 -> /M SW
- L1-->l2Connection1 pad 4: +5V -> /TX
- L1-->l2Connection1 pad 5: +5V -> /RX
- L1-->l2Connection1 pad 6: /M SW -> +5V
- L1-->l2Connection1 pad 7: GND -> +5V
- U1 pad 1: unconnected-(U1-Pad1) -> /Dribbler Data
- U1 pad 11: unconnected-(U1-Pad11) -> /M3 PWM
- U1 pad 12: unconnected-(U1-Pad12) -> /M4 PWM
- U1 pad 2: unconnected-(U1-Pad2) -> /LightGateLDR
- U1 pad 3: unconnected-(U1-Pad3) -> /M3 IN A
- U1 pad 4: unconnected-(U1-Pad4) -> /M3 IN B
- U1 pad 5: unconnected-(U1-Pad5) -> /M4 IN A
- U1 pad 6: unconnected-(U1-Pad6) -> /M4 IN B
Routing:
- net /M2 IN B: track 128.7 -> 68.8 mm
- net /M2 PWM: track 123.7 -> 103.4 mm
