File: elec/layer1/layer1.kicad_pcb (KiCad board)
At the start: 2 copper layers, 178 x 173.3 mm, 115 parts, among them U1 DEV-15583, U2 CD74HC4067SM, U3 CD74HC4067SM

Commit message: l1 half motors done
Parts:
- removed L1-->L2Connection2: Conn_01x08, L1:PinHeader_1x08_P2.54mm_Vertical
- Driver5, Driver6, Driver7, Driver8: footprint Pinheaders:PinHeader_1x08_P2.54mm_Vertical -> Connector_JST:JST_XH_B8B-XH-A_1x08_P2.50mm_Vertical
- moved Driver7 231.4 mm to (277.6, 128.8), turned to 180 degrees
- moved Driver8 219.4 mm to (260.0, 177.4)
- moved Driver6 103.9 mm to (120.0, 177.4)
- moved L1-->l2Connection1 31.7 mm to (188.1, 72.0), turned to 90 degrees
- moved Driver5 18.0 mm to (137.8, 129.0), turned to 180 degrees
Connections:
- Driver5 pad 6: /M SW3 -> /M SW
- Driver7 pad 3: /M2 PWM -> /M4 PWM
- Driver7 pad 7: /M2 IN A -> /M4 IN A
- L1-->l2Connection1 pad 1: /Dribbler Data -> /LightGateLDR
- L1-->l2Connection1 pad 2: /LightGateLDR -> /Dribbler Data
- L1-->l2Connection1 pad 4: /TX -> /RX
- L1-->l2Connection1 pad 5: /RX -> /TX
- L1-->l2Connection1 pad 6: +5V -> /Sol
- L1-->l2Connection1 pad 8: GND -> +5V
- U1 pad 0: /M2 IN B -> /Dribbler Data
- U1 pad 1: /Dribbler Data -> /LightGateLDR
- U1 pad 10: /M2 PWM -> /M1 PWM
- U1 pad 11: /M3 PWM -> /M2 PWM
- U1 pad 12: /M4 PWM -> /M3 PWM
- U1 pad 2: /LightGateLDR -> /M4 IN A
- U1 pad 3: /M3 IN A -> /M4 IN B
- U1 pad 4: /M3 IN B -> /M2 IN B
- U1 pad 5: /M4 IN A -> /M3 IN A
- U1 pad 6: /M4 IN B -> /M3 IN B
- U1 pad 9: /M1 PWM -> /M4 PWM
Routing:
- net /M3 IN A: track 0.00 -> 150.5 mm, vias 0 -> 1
- net /M3 IN B: track 0.00 -> 131.9 mm, vias 0 -> 1
- net +12V: track 254.4 -> 154.9 mm, vias 1 -> 0
- net /M2 IN B: track 68.8 -> 151.6 mm, vias 1 -> 4
- net /M3 PWM: track 0.00 -> 76.3 mm
- net /M SW: track 248.3 -> 172.7 mm, vias 2 -> 1
- net /Sol: track 0.00 -> 60.1 mm, vias 0 -> 1
- net /M1 PWM: track 120.9 -> 66.7 mm, vias 0 -> 1
- net /M2 PWM: track 103.4 -> 135.7 mm, vias 0 -> 2
- net /LightGateLDR: track 0.00 -> 26.8 mm
- net /Dribbler Data: track 0.00 -> 26.2 mm
- net +3V3: track 178.4 -> 158.8 mm
- net /M2 IN A: track 109.4 -> 125.6 mm
- net /M1 IN A: track 120.4 -> 112.7 mm
- net +5V: track 36.4 -> 43.9 mm
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- added copper zone on B.Cu, net +12V
- added copper zone on F.Cu, net +12V
Other:
- board text removed: "12v"
- board text removed: "3v3"
- board text removed: "5v"
- board text removed: "Gnd"
- board text removed: "Rx"
- board text removed: "Tx"

Commit message: allah
Routing:
- net /M SW: track 172.7 -> 370.0 mm, vias 1 -> 2
- net /M4 PWM: track 0.00 -> 145.6 mm, vias 0 -> 1
- net /M4 IN B: track 0.00 -> 130.2 mm, vias 0 -> 2
- net /M4 IN A: track 0.00 -> 119.1 mm, vias 0 -> 2
- net /M1 PWM: track 66.7 -> 141.1 mm, vias 1 -> 2
- net /M1 IN A: track 112.7 -> 120.4 mm
- net +3V3: track 158.8 -> 162.4 mm
- net /M1 IN B: track 94.4 -> 97.9 mm
- net +12V: track 154.9 -> 156.8 mm
- net GND: vias 80 -> 86

Commit message: touched l1
Routing:
- net /M2 PWM: track 135.7 -> 136.8 mm
- net GND: vias 86 -> 88

Commit message: er
Parts:
- L1-->l2Connection1: footprint Pinheaders:PinHeader_1x09_P2.54mm_Vertical -> Connector_JST:JST_XH_S9B-XH-A_1x09_P2.50mm_Horizontal

Commit message: l1+l2 added jsts
Parts:
- L1-->l2Connection1: footprint Connector_JST:JST_XH_S9B-XH-A_1x09_P2.50mm_Horizontal -> Connector_JST:JST_XH_B9B-XH-A_1x09_P2.50mm_Vertical
- turned L1-->l2Connection1 to 0 degrees
Routing:
- net +5V: track 43.9 -> 40.1 mm
- net /Sol: track 60.1 -> 57.8 mm
- net /M2 IN B: track 151.6 -> 152.4 mm
- net GND: vias 88 -> 93

Commit message: unfucked bucks and touched on l1/2
Routing:
- net /M SW: track 370.0 -> 372.3 mm
- net GND: vias 93 -> 95
