File: elec/layer3/layer3.kicad_sch (KiCad schematic)
At the start: 0 parts

Commit message: prod: l1-l3
Parts:
- added H1, H2, H3, H4, H5, H6: MountingHole, MountingHole:MountingHole_3.2mm_M3_DIN965_Pad, symbol Mechanical:MountingHole
