File: elec/layer3/layer3.kicad_sch (KiCad schematic)
At the start: 57 parts, among them J10 Conn_01x05, J4 Conn_01x05, J8 XT30PW-M, J9 XT30PW-M, SW1 SW_SPDT_312, SW2 SW_SPDT_312, SW3 SW_SPDT_312, SW4 SW_SPDT_312, U1 CD74HC4067SM, U2 CD74HC4067SM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

Commit message: all layes drc and fixed
Parts:
- removed R5, R7: 10k, Resistor_SMD:R_0603_1608Metric, symbol Device:R
- removed R6, R8: 10uF, Resistor_SMD:R_0603_1608Metric, symbol Device:R
Connections:
- net Mux Com (1-16): now also U5.9 (D8)
- net Mux Com (17-32): now also U5.2 (D1)

Commit message: chore: fix all 3 layers; prod: all 3 layers
Parts:
- removed R1, R33: 3k24, Resistor_SMD:R_0603_1608Metric, symbol Device:R
Connections:
- net +3V3: now also U4.JP1_1 (VIN)
- net +5V: no longer U4.JP1_1 (VIN)
