File: elec/layer3/layer3.kicad_pcb (KiCad board)
At the start: 2 copper layers, 125 x 125 mm, 53 parts, among them J10 Conn_01x05, J4 Conn_01x05, J8 XT30PW-M, J9 XT30PW-M, U1 CD74HC4067SM, U2 CD74HC4067SM, U4 4754, U5 113991054

Commit message: l3 done
Parts:
- moved R33 0.30 mm to (114.9, 85.3)
- moved R43 0.10 mm to (121.7, 98.1)
- moved R1 0.10 mm to (178.1, 97.8)
Connections:
- R33 pad 2: /Mux Com (17-32) -> /Mux Com (1-16)
- U2 pad 1: /Mux Com (17-32) -> /Mux Com (1-16)
- U5 pad 6: /Mux Com (17-32) -> /Mux Com (1-16)
Routing:
- net /RX(ESP32): track 0.00 -> 83.8 mm, vias 0 -> 1
- net /Mux Com (1-16): track 0.00 -> 80.6 mm, vias 0 -> 1
- net /S1: track 31.5 -> 86.0 mm, vias 1 -> 3
- net /Mux Com (17-32): track 93.4 -> 42.4 mm, vias 3 -> 1
- net /TX(ESP32): track 0.00 -> 43.8 mm
- net +3V3: track 52.7 -> 82.1 mm
- net /S3: track 64.5 -> 77.2 mm
- net Net-(U4-P1): track 0.00 -> 3.67 mm
- net Net-(U4-P0): track 0.00 -> 3.65 mm
- net /S2: track 82.9 -> 82.5 mm, vias 4 -> 2
- net GND: vias 2 -> 4

Commit message: l3: moved jsts
Parts:
- moved J10 14.8 mm to (107.3, 68.4)
- moved J4 14.8 mm to (107.3, 76.2)
Routing:
- net /RX(ESP32): track 83.8 -> 99.7 mm, vias 1 -> 2
- net /SCL (IMU): track 35.9 -> 50.6 mm
- net /TX(ESP32): track 43.8 -> 58.2 mm, vias 0 -> 1
- net /RX (CAM): track 38.1 -> 52.4 mm
- net /SDA (IMU): track 36.0 -> 50.1 mm
- net /TX (CAM): track 43.8 -> 55.9 mm
- net /IR1: track 63.3 -> 72.3 mm
- net /IR2: track 53.4 -> 61.8 mm
- net /IR7: track 33.0 -> 31.4 mm
- net /IR6: track 38.0 -> 39.2 mm
- net /IR5: track 38.4 -> 39.5 mm
- net /IR4: track 38.8 -> 39.5 mm

Commit message: l3 touched
Parts:
- removed IR10, IR11, IR12, IR13, IR14, IR15, IR16, IR17, IR18, IR19, IR2, IR20, IR21, IR22, IR23, IR24, IR25, IR26, IR27, IR28, IR29, IR3, IR30, IR31, IR32, IR4, IR5, IR6, IR7, IR8, IR9: TSSP58038, OptoDevice:Vishay_MINICAST-3Pin
- added IR1: TSSP58038, OptoDevice:Vishay_MINICAST-3Pin, F.Cu at (148.8, 42.0)
- added IR33: TSSP58038, OptoDevice:Vishay_MINICAST-3Pin, F.Cu at (137.7, 42.7)
- added IR34: TSSP58038, OptoDevice:Vishay_MINICAST-3Pin, F.Cu at (127.0, 45.7)
- added IR35: TSSP58038, OptoDevice:Vishay_MINICAST-3Pin, F.Cu at (117.2, 50.9)
- added IR36: TSSP58038, OptoDevice:Vishay_MINICAST-3Pin, F.Cu at (108.7, 58.0)
- added IR37: TSSP58038, OptoDevice:Vishay_MINICAST-3Pin, F.Cu at (101.8, 66.7)
- added IR38: TSSP58038, OptoDevice:Vishay_MINICAST-3Pin, F.Cu at (97.0, 76.7)
- added IR39: TSSP58038, OptoDevice:Vishay_MINICAST-3Pin, F.Cu at (94.2, 87.4)
- added IR40: TSSP58038, OptoDevice:Vishay_MINICAST-3Pin, F.Cu at (93.8, 98.5)
- added IR41: TSSP58038, OptoDevice:Vishay_MINICAST-3Pin, F.Cu at (95.7, 109.4)
- added IR42: TSSP58038, OptoDevice:Vishay_MINICAST-3Pin, F.Cu at (99.8, 119.7)
- added IR43: TSSP58038, OptoDevice:Vishay_MINICAST-3Pin, F.Cu at (106.0, 129.0)
- added IR44: TSSP58038, OptoDevice:Vishay_MINICAST-3Pin, F.Cu at (113.9, 136.7)
- added IR45: TSSP58038, OptoDevice:Vishay_MINICAST-3Pin, F.Cu at (123.3, 142.6)
- added IR46: TSSP58038, OptoDevice:Vishay_MINICAST-3Pin, F.Cu at (133.7, 146.4)
- added IR47: TSSP58038, OptoDevice:Vishay_MINICAST-3Pin, F.Cu at (144.7, 148.0)
- added IR48: TSSP58038, OptoDevice:Vishay_MINICAST-3Pin, F.Cu at (155.8, 147.3)
- added IR49: TSSP58038, OptoDevice:Vishay_MINICAST-3Pin, F.Cu at (166.5, 144.3)
- added IR50: TSSP58038, OptoDevice:Vishay_MINICAST-3Pin, F.Cu at (176.3, 139.1)
- added IR51: TSSP58038, OptoDevice:Vishay_MINICAST-3Pin, F.Cu at (184.8, 132.0)
- added IR52: TSSP58038, OptoDevice:Vishay_MINICAST-3Pin, F.Cu at (191.7, 123.3)
- added IR53: TSSP58038, OptoDevice:Vishay_MINICAST-3Pin, F.Cu at (196.5, 113.3)
- added IR54: TSSP58038, OptoDevice:Vishay_MINICAST-3Pin, F.Cu at (199.3, 102.6)
- added IR55: TSSP58038, OptoDevice:Vishay_MINICAST-3Pin, F.Cu at (199.7, 91.5)
- added IR56: TSSP58038, OptoDevice:Vishay_MINICAST-3Pin, F.Cu at (197.8, 80.6)
- added IR57: TSSP58038, OptoDevice:Vishay_MINICAST-3Pin, F.Cu at (193.7, 70.3)
- added IR58: TSSP58038, OptoDevice:Vishay_MINICAST-3Pin, F.Cu at (187.5, 61.0)
- added IR59: TSSP58038, OptoDevice:Vishay_MINICAST-3Pin, F.Cu at (179.6, 53.3)
- added IR60: TSSP58038, OptoDevice:Vishay_MINICAST-3Pin, F.Cu at (170.2, 47.4)
- added SW1: SW_SPDT_312, L3:SS12D00G3, F.Cu at (148.3, 55.0)
- added SW2: SW_SPDT_312, L3:SS12D00G3, F.Cu at (152.2, 55.0)
- added SW3: SW_SPDT_312, L3:SS12D00G3, F.Cu at (155.9, 55.0)
- added SW4: SW_SPDT_312, L3:SS12D00G3, F.Cu at (159.7, 55.0)
- J8, J9: moved to B.Cu
- moved H1 45.0 mm to (169.1, 55.0)
- moved H2 45.0 mm to (124.1, 55.0)
- moved H3 45.0 mm to (169.1, 135.0)
- moved H4 45.0 mm to (124.1, 135.0)
- moved IR61 11.1 mm to (159.8, 43.6), turned to 168 degrees
- turned J8 to 180 degrees
- turned J9 to 180 degrees
- renumbered IR1 to IR61
Connections:
- IR61 pad 1: /IR1 -> /IR30
- U1 pad 16: /IR32 -> /Strat2
- U1 pad 17: /IR31 -> /IR30
- U1 pad 18: /IR30 -> /IR29
- U1 pad 19: /IR29 -> /IR28
- U1 pad 2: /IR24 -> /IR23
- U1 pad 20: /IR28 -> /IR27
- U1 pad 21: /IR27 -> /IR26
- U1 pad 22: /IR26 -> /IR25
- U1 pad 23: /IR25 -> /IR24
- U1 pad 3: /IR23 -> /IR22
- U1 pad 4: /IR22 -> /IR21
- U1 pad 5: /IR21 -> /IR20
- U1 pad 6: /IR20 -> /IR19
- U1 pad 7: /IR19 -> /IR18
- U1 pad 8: /IR18 -> /IR17
- U1 pad 9: /IR17 -> /IR16
- U2 pad 16: /IR16 -> /Strat1
- U5 pad 10: unconnected-(U5-D9-Pad10) -> /Strat4
- U5 pad 9: unconnected-(U5-D8-Pad9) -> /Strat3
Routing:
- net /Strat1: track 0.00 -> 57.4 mm, vias 0 -> 2
- net /IR32: track 50.1 -> 0.00 mm
- net /Strat2: track 0.00 -> 46.4 mm
- net /IR31: track 42.8 -> 0.00 mm
- net /Strat3: track 0.00 -> 39.0 mm
- net /Strat4: track 0.00 -> 33.2 mm
- net /IR16: track 56.8 -> 73.5 mm
- net +3V3: track 82.1 -> 98.0 mm, vias 2 -> 1
- net /IR1: track 72.3 -> 58.0 mm
- net /IR30: track 37.4 -> 49.9 mm
- net +5V: track 111.3 -> 122.6 mm
- net /IR23: track 40.0 -> 29.2 mm
- net /IR17: track 68.5 -> 59.6 mm
- net /IR2: track 61.8 -> 53.0 mm
- net /IR19: track 53.7 -> 44.9 mm
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
Commit message: fix: l3
Parts:
- moved J8 85.8 mm to (102.3, 106.5), turned to -90 degrees
- moved J9 5.61 mm to (102.3, 91.0), turned to -90 degrees
Routing:
- net +5V: track 122.6 -> 135.1 mm, vias 1 -> 0
- net /IR10: track 32.1 -> 38.4 mm
- net +3V3: track 98.0 -> 100.4 mm, vias 1 -> 0
- net GND: vias 4 -> 1
Other:
- board text added: "0"
- board text added: "1"
- board text added: "3v3"
- board text added: "5v"
- board text added: "GOAL"
- board text added: "L2"
- board text added: "SIDE"
- board text added: "Vent Exhaust"

Commit message: prod: l2, l3
Parts:
- moved U6 28.7 mm to (146.6, 109.4)
Routing:
- net +5V: track 135.1 -> 142.3 mm
- net /TX (CAM): track 56.4 -> 56.6 mm, vias 0 -> 1
Other:
- outline, holes or cut-outs redrawn
