File: elec/layer2/motor.kicad_sch (KiCad schematic)
At the start: 12 parts, among them Q1 AON6354, U2 VNH5019ATR-E, U3 XT30UPB-M

Commit message: feat: l2 schematics
Parts:
- removed U3: XT30UPB-M, Connector_AMASS:AMASS_XT30UPB-M_1x02_P5.0mm_Vertical, symbol amass xt 30:XT30UPB-M
- added J13: XT30PW-M, layer2-pcb-footprints:AMASS_XT30PW-M, symbol layer2-pcb-symbols:XT30PW-M
- added TP12, TP4, TP8: TestPoint, symbol Connector:TestPoint
Connections:
- net Motor IN A: now also TP4.1
- net Motor IN B: now also TP8.1
- net Motor Out A: now also J13.N
- net Motor Out B: now also J13.P
- net Motor PWM: now also TP12.1

Commit message: feat: buck.steps; chore: l2
Parts:
- Q1: footprint initium20:8-DFN (5x6) -> layer2-pcb-footprints:8-DFN (5x6)
- TP12, TP4, TP8: footprint (none) -> TestPoint:TestPoint_THTPad_D1.5mm_Drill0.7mm
Changed lines of the file:
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@@
 			)
 		)
-		(property "Footprint" ""
+		(property "Footprint" "TestPoint:TestPoint_THTPad_D1.5mm_Drill0.7mm"
 			(at 95.25 97.79 0)
 			(effects
@@
 			)
 		)
-		(property "Footprint" "initium20:8-DFN (5x6)"
+		(property "Footprint" "layer2-pcb-footprints:8-DFN (5x6)"
 			(at 191.77 78.74 90)
 			(effects
@@
 			)
 		)
-		(property "Footprint" ""
+		(property "Footprint" "TestPoint:TestPoint_THTPad_D1.5mm_Drill0.7mm"
 			(at 95.25 92.71 0)
 			(effects
@@
 			)
 		)
-		(property "Footprint" ""
+		(property "Footprint" "TestPoint:TestPoint_THTPad_D1.5mm_Drill0.7mm"
 			(at 95.25 105.41 0)
 			(effects
