File: elec/layer2/layer2.kicad_pcb (KiCad board)
At the start: 2 copper layers, 178 x 173.3 mm, 0 parts

Commit message: fix: l1 gnd
Parts:
- added C1: 470u, Capacitor_THT:CP_Radial_D8.0mm_P3.50mm, F.Cu at (217.4, 181.2)
- added C2: 470u, Capacitor_THT:CP_Radial_D8.0mm_P3.50mm, F.Cu at (232.2, 181.2)
- added C3: 470u, Capacitor_THT:CP_Radial_D8.0mm_P3.50mm, F.Cu at (259.3, 169.7)
- added C4: 470u, Capacitor_THT:CP_Radial_D8.0mm_P3.50mm, F.Cu at (245.1, 141.4)
- added C9: 470u, Capacitor_THT:CP_Radial_D8.0mm_P3.50mm, F.Cu at (71.5, 172.8)
- added J2: XT30UPB-M, layer2-pcb-footprints:AMASS_XT30UPB-M, F.Cu at (228.6, 121.2)
- added Q1: AON6354, initium20:8-DFN (5x6), F.Cu at (77.3, 153.9)
- added R1: 3K3, Resistor_SMD:R_0603_1608Metric, F.Cu at (225.0, 158.9)
- added R10: 3K3, Resistor_SMD:R_0603_1608Metric, F.Cu at (77.0, 164.9)
- added R11: 10K, Resistor_SMD:R_0603_1608Metric, F.Cu at (77.0, 167.9)
- added R12: 1K, Resistor_SMD:R_0603_1608Metric, F.Cu at (77.0, 163.4)
- added R13: 1K, Resistor_SMD:R_0603_1608Metric, F.Cu at (77.0, 169.4)
- added R14: 1K, Resistor_SMD:R_0603_1608Metric, F.Cu at (77.0, 161.9)
- added R15: 1K, Resistor_SMD:R_0603_1608Metric, F.Cu at (77.0, 166.4)
- added R16: 1K, Resistor_SMD:R_0603_1608Metric, F.Cu at (240.8, 177.7)
- added R17: 3K3, Resistor_SMD:R_0603_1608Metric, F.Cu at (254.1, 158.9)
- added R18: 3K3, Resistor_SMD:R_0603_1608Metric, F.Cu at (254.1, 161.4)
- added R19: 10K, Resistor_SMD:R_0603_1608Metric, F.Cu at (254.1, 163.9)
- added R2: 3K3, Resistor_SMD:R_0603_1608Metric, F.Cu at (225.0, 161.4)
- added R20: 1K, Resistor_SMD:R_0603_1608Metric, F.Cu at (254.1, 166.4)
- added R21: 1K, Resistor_SMD:R_0603_1608Metric, F.Cu at (254.1, 169.0)
- added R22: 1K, Resistor_SMD:R_0603_1608Metric, F.Cu at (254.1, 171.5)
- added R23: 1K, Resistor_SMD:R_0603_1608Metric, F.Cu at (254.1, 174.0)
- added R24: 1K, Resistor_SMD:R_0603_1608Metric, F.Cu at (254.1, 176.5)
- added R25: 3K3, Resistor_SMD:R_0603_1608Metric, F.Cu at (239.9, 119.1)
- added R26: 3K3, Resistor_SMD:R_0603_1608Metric, F.Cu at (239.9, 121.6)
- added R27: 10K, Resistor_SMD:R_0603_1608Metric, F.Cu at (239.9, 124.1)
- added R28: 1K, Resistor_SMD:R_0603_1608Metric, F.Cu at (239.9, 126.6)
- added R29: 1K, Resistor_SMD:R_0603_1608Metric, F.Cu at (239.9, 129.1)
- added R3: 10K, Resistor_SMD:R_0603_1608Metric, F.Cu at (225.0, 163.9)
- added R30: 1K, Resistor_SMD:R_0603_1608Metric, F.Cu at (239.9, 131.7)
- added R31: 1K, Resistor_SMD:R_0603_1608Metric, F.Cu at (239.9, 134.2)
- added R32: 1K, Resistor_SMD:R_0603_1608Metric, F.Cu at (239.9, 136.7)
- added R4: 1K, Resistor_SMD:R_0603_1608Metric, F.Cu at (225.0, 166.4)
- added R5: 1K, Resistor_SMD:R_0603_1608Metric, F.Cu at (225.0, 169.0)
- added R6: 1K, Resistor_SMD:R_0603_1608Metric, F.Cu at (225.0, 171.5)
- added R7: 1K, Resistor_SMD:R_0603_1608Metric, F.Cu at (225.0, 174.0)
- added R8: 1K, Resistor_SMD:R_0603_1608Metric, F.Cu at (77.0, 160.4)
- added R9: 3K3, Resistor_SMD:R_0603_1608Metric, F.Cu at (77.0, 170.9)
- added SW1: SW_SPDT_312, layer2-pcb-footprints:SS12D00G3, F.Cu at (226.2, 126.9)
- added TP1: TestPoint_2Pole, TestPoint:TestPoint_2Pads_Pitch2.54mm_Drill0.8mm, F.Cu at (223.1, 131.0)
- added TP2: TestPoint_2Pole, TestPoint:TestPoint_2Pads_Pitch2.54mm_Drill0.8mm, F.Cu at (223.1, 134.3)
- added U1: TEENSY40, layer2-pcb-footprints:TEENSY40, F.Cu at (211.6, 137.1)
- added U2: VNH5019ATR-E, layer2-pcb-footprints:VNH5019ATR-E, F.Cu at (212.5, 167.0)
- added U3: XT30UPB-M, Connector_AMASS:AMASS_XT30UPB-M_1x02_P5.0mm_Vertical, F.Cu at (205.6, 180.0)
- added U4: VNH5019ATR-E, layer2-pcb-footprints:VNH5019ATR-E, F.Cu at (239.5, 167.0)
- added U5: XT30UPB-M, initium20:VNH5019ATR-E, F.Cu at (63.8, 160.8)
- added U6: VNH5019ATR-E, Connector_AMASS:AMASS_XT30UPB-M_1x02_P5.0mm_Vertical, F.Cu at (57.2, 174.7)
- added U7: XT30UPB-M, Connector_AMASS:AMASS_XT30UPB-M_1x02_P5.0mm_Vertical, F.Cu at (259.7, 161.3)
- added U8: VNH5019ATR-E, layer2-pcb-footprints:VNH5019ATR-E, F.Cu at (252.4, 127.2)
- added U9: XT30UPB-M, Connector_AMASS:AMASS_XT30UPB-M_1x02_P5.0mm_Vertical, F.Cu at (255.3, 140.2)
Routing:
- net Net-(Q1-G): track 0.00 -> 7.17 mm, vias 0 -> 2
- net Net-(U4-ENB/DIAGB): track 0.00 -> 6.53 mm
- net Net-(U4-INB): track 0.00 -> 6.20 mm
- net GND: track 0.00 -> 5.89 mm
- net Net-(U4-INA): track 0.00 -> 5.50 mm
- net Net-(U4-ENA/DIAGA): track 0.00 -> 5.11 mm
- net /Motor 1 PWM: track 0.00 -> 1.50 mm
- net /Motor 1 IN B: track 0.00 -> 1.50 mm
- net Net-(C1-Pad1): vias 0 -> 5
- net /Motor 2/Motor Out B: vias 0 -> 1
- net /Motor 1/Motor Out A: vias 0 -> 14
- added copper zone on F.Cu, net +12V
- added copper zone on B.Cu, net /Motor 1/Motor Out A
- added copper zone on F.Cu, net /Motor 1/Motor Out A
- added copper zone on B.Cu, net /Motor 1/Motor Out B
- added copper zone on F.Cu, net /Motor 1/Motor Out B
- added copper zone on B.Cu, net Net-(C1-Pad1)
- added copper zone on F.Cu, net Net-(C1-Pad1)
Other:
- board outline removed

Commit message: feat: l2 schematics
Parts:
- removed C1, C2, C3, C4, C9: 470u, Capacitor_THT:CP_Radial_D8.0mm_P3.50mm
- removed J2: XT30UPB-M, layer2-pcb-footprints:AMASS_XT30UPB-M
- removed Q1: AON6354, initium20:8-DFN (5x6)
- removed R1, R10, R17, R18, R2, R25, R26, R9: 3K3, Resistor_SMD:R_0603_1608Metric
- removed R11, R19, R27, R3: 10K, Resistor_SMD:R_0603_1608Metric
- removed R12, R13, R14, R15, R16, R20, R21, R22, R23, R24, R28, R29, R30, R31, R32, R4, R5, R6, R7, R8: 1K, Resistor_SMD:R_0603_1608Metric
- removed SW1: SW_SPDT_312, layer2-pcb-footprints:SS12D00G3
- removed TP1, TP2: TestPoint_2Pole, TestPoint:TestPoint_2Pads_Pitch2.54mm_Drill0.8mm
- removed U1: TEENSY40, layer2-pcb-footprints:TEENSY40
- removed U2, U4, U8: VNH5019ATR-E, layer2-pcb-footprints:VNH5019ATR-E
- removed U3, U7, U9: XT30UPB-M, Connector_AMASS:AMASS_XT30UPB-M_1x02_P5.0mm_Vertical
- removed U5: XT30UPB-M, initium20:VNH5019ATR-E
- removed U6: VNH5019ATR-E, Connector_AMASS:AMASS_XT30UPB-M_1x02_P5.0mm_Vertical
Routing:
- net Net-(Q1-G): track 7.17 -> 0.00 mm, vias 2 -> 0
- net Net-(U4-ENB/DIAGB): track 6.53 -> 0.00 mm
- net Net-(U4-INB): track 6.20 -> 0.00 mm
- net GND: track 5.89 -> 0.00 mm
- net Net-(U4-INA): track 5.50 -> 0.00 mm
- net Net-(U4-ENA/DIAGA): track 5.11 -> 0.00 mm
- net /Motor 1 PWM: track 1.50 -> 0.00 mm
- net /Motor 1 IN B: track 1.50 -> 0.00 mm
- net Net-(C1-Pad1): vias 5 -> 0
- net /Motor 2/Motor Out B: vias 1 -> 0
- net /Motor 1/Motor Out A: vias 14 -> 0
- added copper zone on B.Cu, net GND
- added copper zone on F.Cu, net GND
- removed copper zone on F.Cu, net +12V
- removed copper zone on B.Cu, net /Motor 1/Motor Out A
- removed copper zone on F.Cu, net /Motor 1/Motor Out A
- removed copper zone on B.Cu, net /Motor 1/Motor Out B
- removed copper zone on F.Cu, net /Motor 1/Motor Out B
- removed copper zone on B.Cu, net Net-(C1-Pad1)
- removed copper zone on F.Cu, net Net-(C1-Pad1)
Other:
- board outline added: 178 x 173.3 mm
- board text added: "buck (back)"
- board text added: "dribbler connections"
- board text added: "kicker"
- board text added: "motor drivers"
- board text added: "motor xt30s"
- board text added: "teensy"

Commit message: feat: buck.steps; chore: l2
Parts:
- added C1: 470u, Capacitor_THT:CP_Radial_D8.0mm_P3.50mm, B.Cu at (82.0, 120.4)
- added C2: 470u, Capacitor_THT:CP_Radial_D8.0mm_P3.50mm, B.Cu at (107.2, 120.1)
- added C3: 470u, Capacitor_THT:CP_Radial_D8.0mm_P3.50mm, B.Cu at (134.0, 119.8)
- added C4: 470u, Capacitor_THT:CP_Radial_D8.0mm_P3.50mm, B.Cu at (159.2, 119.9)
- added H1: MountingHole, MountingHole:MountingHole_3.2mm_M3_DIN965_Pad, F.Cu at (79.6, 30.1)
- added H10: MountingHole, MountingHole:MountingHole_3.2mm_M3_DIN965_Pad, F.Cu at (189.8, 140.3)
- added H11: MountingHole, MountingHole:MountingHole_3.2mm_M3_DIN965_Pad, F.Cu at (81.6, 181.6)
- added H12: MountingHole, MountingHole:MountingHole_3.2mm_M3_DIN965_Pad, F.Cu at (147.4, 181.6)
- added H2: MountingHole, MountingHole:MountingHole_3.2mm_M3_DIN965_Pad, F.Cu at (149.4, 30.1)
- added H3: MountingHole, MountingHole:MountingHole_3.2mm_M3_DIN965_Pad, F.Cu at (39.2, 70.6)
- added H4: MountingHole, MountingHole:MountingHole_3.2mm_M3_DIN965_Pad, F.Cu at (189.8, 70.6)
- added H5: MountingHole, MountingHole:MountingHole_3.2mm_M3_DIN965_Pad, F.Cu at (74.5, 82.9)
- added H6: MountingHole, MountingHole:MountingHole_3.2mm_M3_DIN965_Pad, F.Cu at (154.5, 82.9)
- added H7: MountingHole, MountingHole:MountingHole_3.2mm_M3_DIN965_Pad, F.Cu at (74.5, 127.9)
- added H8: MountingHole, MountingHole:MountingHole_3.2mm_M3_DIN965_Pad, F.Cu at (154.5, 127.9)
- added H9: MountingHole, MountingHole:MountingHole_3.2mm_M3_DIN965_Pad, F.Cu at (39.2, 140.3)
- added J1: Conn_01x03, Connector_JST:JST_XH_B3B-XH-A_1x03_P2.50mm_Vertical, F.Cu at (2.98, 2.88)
- added J10: Conn_01x05, Connector_JST:JST_XH_B5B-XH-A_1x05_P2.50mm_Vertical, F.Cu at (3.42, 62.7)
- added J11: Conn_01x05, Connector_JST:JST_XH_B5B-XH-A_1x05_P2.50mm_Vertical, F.Cu at (8.01, 62.7)
- added J12: XT60-M, layer2-pcb-footprints:AMASS_XT60-M, F.Cu at (39.8, 118.7)
- added J13: XT30PW-M, layer2-pcb-footprints:AMASS_XT30PW-M, B.Cu at (174.5, 88.4)
- added J14: XT30PW-M, layer2-pcb-footprints:AMASS_XT30PW-M, B.Cu at (189.5, 88.4)
- added J15: XT30PW-M, layer2-pcb-footprints:AMASS_XT30PW-M, B.Cu at (174.5, 122.4)
- added J16: XT30PW-M, layer2-pcb-footprints:AMASS_XT30PW-M, B.Cu at (189.5, 122.4)
- added J17: Conn_01x02, Connector_JST:JST_XH_B2B-XH-A_1x02_P2.50mm_Vertical, F.Cu at (4.68, 45.7)
- added J18: Conn_01x02, Connector_JST:JST_XH_B2B-XH-A_1x02_P2.50mm_Vertical, F.Cu at (9.27, 45.7)
- added J2: XT30UPB-M, layer2-pcb-footprints:AMASS_XT30UPB-M, F.Cu at (3.85, 78.6)
- added J3: Conn_01x04, Connector_JST:JST_XH_B4B-XH-A_1x04_P2.50mm_Vertical, F.Cu at (-5.61, 102.6)
- added J4: Conn_01x05, Connector_JST:JST_XH_B5B-XH-A_1x05_P2.50mm_Vertical, F.Cu at (-1.17, 62.7)
- added J5: Conn_01x03, Connector_JST:JST_XH_B3B-XH-A_1x03_P2.50mm_Vertical, F.Cu at (2.98, 10.7)
- added J6: XT30PW-M, layer2-pcb-footprints:AMASS_XT30PW-M, B.Cu at (55.3, 120.6)
- added J7: XT30PW-M, layer2-pcb-footprints:AMASS_XT30PW-M, F.Cu at (-26.2, 66.7)
- added J8: XT30PW-M, layer2-pcb-footprints:AMASS_XT30PW-M, F.Cu at (11.3, 127.1)
- added J9: XT30PW-M, layer2-pcb-footprints:AMASS_XT30PW-M, F.Cu at (-5.04, 47.1)
- added KillSwitch2: SW_SPST, layer2-pcb-footprints:AMASS_XT30UPB-M, F.Cu at (39.3, 110.9)
- added Q1: AON6354, layer2-pcb-footprints:8-DFN (5x6), B.Cu at (84.0, 90.4)
- added Q2: AON6354, layer2-pcb-footprints:8-DFN (5x6), B.Cu at (109.2, 90.1)
- added Q3: AON6354, layer2-pcb-footprints:8-DFN (5x6), B.Cu at (136.0, 89.8)
- added Q4: AON6354, layer2-pcb-footprints:8-DFN (5x6), B.Cu at (161.2, 89.9)
- added R1: 3K3, Resistor_SMD:R_0603_1608Metric, B.Cu at (78.3, 91.5)
- added R10: 3K3, Resistor_SMD:R_0603_1608Metric, B.Cu at (92.9, 91.2)
- added R11: 10K, Resistor_SMD:R_0603_1608Metric, B.Cu at (97.4, 91.2)
- added R12: 1K, Resistor_SMD:R_0603_1608Metric, B.Cu at (95.9, 91.2)
- added R13: 1K, Resistor_SMD:R_0603_1608Metric, B.Cu at (100.4, 91.2)
- added R14: 1K, Resistor_SMD:R_0603_1608Metric, B.Cu at (94.4, 91.2)
- added R15: 1K, Resistor_SMD:R_0603_1608Metric, B.Cu at (101.9, 91.2)
- added R16: 1K, Resistor_SMD:R_0603_1608Metric, B.Cu at (98.9, 91.2)
- added R17: 3K3, Resistor_SMD:R_0603_1608Metric, B.Cu at (130.3, 90.9)
- added R18: 3K3, Resistor_SMD:R_0603_1608Metric, B.Cu at (119.8, 90.9)
- added R19: 10K, Resistor_SMD:R_0603_1608Metric, B.Cu at (124.3, 90.9)
- added R2: 3K3, Resistor_SMD:R_0603_1608Metric, B.Cu at (67.8, 91.5)
- added R20: 1K, Resistor_SMD:R_0603_1608Metric, B.Cu at (122.8, 90.9)
- added R21: 1K, Resistor_SMD:R_0603_1608Metric, B.Cu at (127.3, 90.9)
- added R22: 1K, Resistor_SMD:R_0603_1608Metric, B.Cu at (121.3, 90.9)
- added R23: 1K, Resistor_SMD:R_0603_1608Metric, B.Cu at (128.8, 90.9)
- added R24: 1K, Resistor_SMD:R_0603_1608Metric, B.Cu at (125.8, 90.9)
- added R25: 3K3, Resistor_SMD:R_0603_1608Metric, B.Cu at (155.5, 91.0)
- added R26: 3K3, Resistor_SMD:R_0603_1608Metric, B.Cu at (145.0, 91.0)
- added R27: 10K, Resistor_SMD:R_0603_1608Metric, B.Cu at (149.5, 91.0)
- added R28: 1K, Resistor_SMD:R_0603_1608Metric, B.Cu at (148.0, 91.0)
- added R29: 1K, Resistor_SMD:R_0603_1608Metric, B.Cu at (152.5, 91.0)
- added R3: 10K, Resistor_SMD:R_0603_1608Metric, B.Cu at (72.3, 91.5)
- added R30: 1K, Resistor_SMD:R_0603_1608Metric, B.Cu at (146.5, 91.0)
- added R31: 1K, Resistor_SMD:R_0603_1608Metric, B.Cu at (154.0, 91.0)
- added R32: 1K, Resistor_SMD:R_0603_1608Metric, B.Cu at (151.0, 91.0)
- added R33: 10k, Resistor_SMD:R_0603_1608Metric, F.Cu at (13.5, 0.76)
- added R4: 1K, Resistor_SMD:R_0603_1608Metric, B.Cu at (70.8, 91.5)
- added R5: 1K, Resistor_SMD:R_0603_1608Metric, B.Cu at (75.3, 91.5)
- added R6: 1K, Resistor_SMD:R_0603_1608Metric, B.Cu at (69.3, 91.5)
- added R7: 1K, Resistor_SMD:R_0603_1608Metric, B.Cu at (76.8, 91.5)
- added R8: 1K, Resistor_SMD:R_0603_1608Metric, B.Cu at (73.8, 91.5)
- added R9: 3K3, Resistor_SMD:R_0603_1608Metric, B.Cu at (103.4, 91.2)
- added SW1: SW_SPDT_312, layer2-pcb-footprints:SS12D00G3, F.Cu at (141.8, 30.7)
- added TP1: TestPoint_2Pole, TestPoint:TestPoint_2Pads_Pitch2.54mm_Drill0.8mm, F.Cu at (7.19, 100.9)
- added TP10: TestPoint, TestPoint:TestPoint_THTPad_D1.5mm_Drill0.7mm, F.Cu at (121.3, 41.7)
- added TP11: TestPoint, TestPoint:TestPoint_THTPad_D1.5mm_Drill0.7mm, F.Cu at (128.8, 41.7)
- added TP12: TestPoint, TestPoint:TestPoint_THTPad_D1.5mm_Drill0.7mm, F.Cu at (103.5, 41.7)
- added TP13: TestPoint, TestPoint:TestPoint_THTPad_D1.5mm_Drill0.7mm, F.Cu at (111.0, 41.7)
- added TP14: TestPoint, TestPoint:TestPoint_THTPad_D1.5mm_Drill0.7mm, F.Cu at (118.8, 41.7)
- added TP15: TestPoint, TestPoint:TestPoint_THTPad_D1.5mm_Drill0.7mm, F.Cu at (126.3, 41.7)
- added TP16: TestPoint, TestPoint:TestPoint_THTPad_D1.5mm_Drill0.7mm, F.Cu at (-55.2, 100.0)
- added TP17: TestPoint, TestPoint:TestPoint_THTPad_D1.5mm_Drill0.7mm, F.Cu at (-55.2, 103.6)
- added TP18: TestPoint, TestPoint:TestPoint_THTPad_D1.5mm_Drill0.7mm, F.Cu at (-55.2, 107.1)
- added TP19: TestPoint, TestPoint:TestPoint_THTPad_D1.5mm_Drill0.7mm, F.Cu at (-51.7, 100.0)
- added TP2: TestPoint_2Pole, TestPoint:TestPoint_2Pads_Pitch2.54mm_Drill0.8mm, F.Cu at (7.19, 104.2)
- added TP20: TestPoint, TestPoint:TestPoint_THTPad_D1.5mm_Drill0.7mm, F.Cu at (-51.7, 103.6)
- added TP21: TestPoint, TestPoint:TestPoint_THTPad_D1.5mm_Drill0.7mm, F.Cu at (-51.7, 107.1)
- added TP22: TestPoint, TestPoint:TestPoint_THTPad_D1.5mm_Drill0.7mm, F.Cu at (-48.1, 100.0)
- added TP23: TestPoint, TestPoint:TestPoint_THTPad_D1.5mm_Drill0.7mm, F.Cu at (-48.1, 103.6)
- added TP24: TestPoint, TestPoint:TestPoint_THTPad_D1.5mm_Drill0.7mm, F.Cu at (-48.1, 107.1)
- added TP25: TestPoint, TestPoint:TestPoint_THTPad_D1.5mm_Drill0.7mm, F.Cu at (-44.6, 100.0)
- added TP26: TestPoint, TestPoint:TestPoint_THTPad_D1.5mm_Drill0.7mm, F.Cu at (-44.6, 103.6)
- added TP27: TestPoint, TestPoint:TestPoint_THTPad_D1.5mm_Drill0.7mm, F.Cu at (-44.6, 107.1)
- added TP28: TestPoint_2Pole, TestPoint:TestPoint_2Pads_Pitch2.54mm_Drill0.8mm, F.Cu at (7.19, 110.9)
- added TP3: TestPoint_2Pole, TestPoint:TestPoint_2Pads_Pitch2.54mm_Drill0.8mm, F.Cu at (7.19, 107.6)
- added TP4: TestPoint, TestPoint:TestPoint_THTPad_D1.5mm_Drill0.7mm, F.Cu at (101.0, 41.7)
- added TP5: TestPoint, TestPoint:TestPoint_THTPad_D1.5mm_Drill0.7mm, F.Cu at (108.5, 41.7)
- added TP6: TestPoint, TestPoint:TestPoint_THTPad_D1.5mm_Drill0.7mm, F.Cu at (116.3, 41.7)
- added TP7: TestPoint, TestPoint:TestPoint_THTPad_D1.5mm_Drill0.7mm, F.Cu at (123.8, 41.7)
- added TP8: TestPoint, TestPoint:TestPoint_THTPad_D1.5mm_Drill0.7mm, F.Cu at (106.0, 41.7)
- added TP9: TestPoint, TestPoint:TestPoint_THTPad_D1.5mm_Drill0.7mm, F.Cu at (113.5, 41.7)
- added U1: TEENSY40, layer2-pcb-footprints:TEENSY40, F.Cu at (114.9, 30.8)
- added U2: VNH5019ATR-E, layer2-pcb-footprints:VNH5019ATR-E, B.Cu at (77.3, 104.0)
- added U3: ~, layer2-pcb-footprints:buck-module, F.Cu at (47.5, 91.9)
- added U4: VNH5019ATR-E, layer2-pcb-footprints:VNH5019ATR-E, B.Cu at (102.4, 103.7)
- added U6: VNH5019ATR-E, layer2-pcb-footprints:VNH5019ATR-E, B.Cu at (129.3, 103.4)
- added U8: VNH5019ATR-E, layer2-pcb-footprints:VNH5019ATR-E, B.Cu at (154.5, 103.5)
Routing:
- net /Motors Enable: track 0.00 -> 308.5 mm, vias 0 -> 8
- net /Motor 1/Motor Out A: track 0.00 -> 156.5 mm
- net /Motor 2/Motor Out A: track 0.00 -> 154.7 mm
- net /Motor 1/Motor Out B: track 0.00 -> 128.1 mm
- net /Motor 2/Motor Out B: track 0.00 -> 118.7 mm
- net /Motor 3/Motor Out B: track 0.00 -> 77.2 mm
- net /Motor 3/Motor Out A: track 0.00 -> 73.0 mm
- net /Motor 1 IN A: track 0.00 -> 69.7 mm
- net /Motor 1 PWM: track 0.00 -> 66.5 mm
- net /Motor 4 IN A: track 0.00 -> 66.5 mm
- net /Motor 1 IN B: track 0.00 -> 65.9 mm
- net /Motor 4 IN B: track 0.00 -> 65.5 mm
- net /Motor 2 IN B: track 0.00 -> 62.9 mm
- net /Motor 4 PWM: track 0.00 -> 62.9 mm
- net /Motor 2 IN A: track 0.00 -> 61.5 mm
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- added copper zone on B.Cu, net +12V
- added copper zone on B.Cu, net /Motor 1/Motor Out A
- added copper zone on F.Cu, net /Motor 1/Motor Out A
- added copper zone on B.Cu, net /Motor 1/Motor Out B
- added copper zone on F.Cu, net /Motor 1/Motor Out B
- added copper zone on B.Cu, net /Motor 2/Motor Out A
- added copper zone on F.Cu, net /Motor 2/Motor Out A
- added copper zone on B.Cu, net /Motor 2/Motor Out B
- added copper zone on F.Cu, net /Motor 2/Motor Out B
- added copper zone on B.Cu, net /Motor 3/Motor Out A
- added copper zone on F.Cu, net /Motor 3/Motor Out A
- added copper zone on B.Cu, net /Motor 3/Motor Out B
- added copper zone on F.Cu, net /Motor 3/Motor Out B
- added copper zone on B.Cu, net /Motor 4/Motor Out A
- added copper zone on F.Cu, net /Motor 4/Motor Out A
- added copper zone on B.Cu, net /Motor 4/Motor Out B
- added copper zone on F.Cu, net /Motor 4/Motor Out B
- added copper zone on B.Cu, net Net-(C1-Pad1)
- added copper zone on F.Cu, net Net-(C1-Pad1)
- added copper zone on B.Cu, net Net-(C2-Pad1)
- added copper zone on F.Cu, net Net-(C2-Pad1)
- added copper zone on B.Cu, net Net-(C3-Pad1)
- added copper zone on F.Cu, net Net-(C3-Pad1)
- added copper zone on B.Cu, net Net-(C4-Pad1)
- added copper zone on F.Cu, net Net-(C4-Pad1)
Other:
- outline, holes or cut-outs redrawn
- board text removed: "buck (back)"
- board text removed: "dribbler connections"
- board text removed: "kicker"
- board text removed: "motor drivers"
- board text removed: "motor xt30s"
- board text removed: "teensy"

Commit message: chore: l2
Parts:
- removed J8: XT30PW-M, layer2-pcb-footprints:AMASS_XT30PW-M
- added J19: XT30UPB-M, layer2-pcb-footprints:AMASS_XT30UPB-M, B.Cu at (189.0, 122.4)
- J6: value XT30PW-M -> XT30UPB-M; footprint layer2-pcb-footprints:AMASS_XT30PW-M -> layer2-pcb-footprints:AMASS_XT30UPB-M
- J7: value XT30PW-M -> XT30UPB-M; footprint layer2-pcb-footprints:AMASS_XT30PW-M -> layer2-pcb-footprints:AMASS_XT30UPB-M; moved to B.Cu
- moved J7 220.9 mm to (189.0, 116.4), turned to 180 degrees
- moved J9 199.9 mm to (190.0, 90.7), turned to 180 degrees
- moved J6 134.0 mm to (189.0, 128.4)
- moved J13 92.7 mm to (83.5, 106.0)
- moved J14 76.5 mm to (115.0, 105.7)
- moved J15 32.6 mm to (146.5, 105.7), turned to 0 degrees
- moved J16 20.3 mm to (178.0, 105.7), turned to 0 degrees
- moved R2 9.52 mm to (58.3, 91.9)
- moved R3 9.52 mm to (62.8, 91.9)
- moved R4 9.52 mm to (61.3, 91.9)
- moved R6 9.52 mm to (59.8, 91.9)
- moved C1 9.52 mm to (72.5, 120.8)
- moved Q1 9.52 mm to (74.5, 90.8)
- moved R1 9.52 mm to (68.8, 91.9)
- moved R5 9.52 mm to (65.8, 91.9)
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Connections:
- J6 pad P: +3V3 -> +5V
- J7 pad P: +5V -> +12V
Routing:
- net /Motors Enable: track 308.5 -> 28.3 mm, vias 8 -> 0
- net /Motor 1/Motor Out A: track 156.5 -> 0.00 mm
- net /Motor 2/Motor Out A: track 154.7 -> 0.00 mm
- net /Motor 1/Motor Out B: track 128.1 -> 0.00 mm
- net /Motor 2/Motor Out B: track 118.7 -> 0.00 mm
- net /Motor 3/Motor Out B: track 77.2 -> 0.00 mm
- net /Motor 3/Motor Out A: track 73.0 -> 0.00 mm
- net /Motor 4/Motor Out A: track 58.1 -> 0.00 mm
- net /Motor 4/Motor Out B: track 46.7 -> 0.00 mm
- net /Motor 1 IN B: track 65.9 -> 82.9 mm
- net /Motor 1 PWM: track 66.5 -> 80.8 mm
- net /Motor 1 IN A: track 69.7 -> 82.8 mm
- net /Motor 4 PWM: track 62.9 -> 71.0 mm
- net /Motor 4 IN B: track 65.5 -> 72.6 mm
- net /Motor 2 IN B: track 62.9 -> 66.1 mm
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
Commit message: feat: l2, lightgate
Parts:
- moved TP27 196.4 mm to (131.5, 20.2)
- moved TP21 195.8 mm to (123.8, 20.2)
- moved TP23 195.6 mm to (128.8, 20.2)
- moved TP18 192.3 mm to (116.3, 20.2)
- moved TP20 192.0 mm to (121.3, 20.2)
- moved TP22 191.8 mm to (126.3, 20.2)
- moved TP1 190.1 mm to (197.3, 99.9)
- moved TP2 190.1 mm to (197.3, 103.3)
- moved TP28 190.1 mm to (197.3, 110.0)
- moved TP3 190.1 mm to (197.3, 106.6)
- moved TP17 188.4 mm to (113.8, 20.2)
- moved TP19 188.2 mm to (118.8, 20.2)
- moved TP26 186.7 mm to (131.5, 41.7)
- moved TP16 184.6 mm to (111.3, 20.2)
- moved TP24 177.0 mm to (106.0, 20.2)
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Routing:
- net /Motor 4/Motor Out A: track 0.00 -> 60.5 mm
- net /Motor 3/Motor Out A: track 0.00 -> 60.2 mm
- net /Motor 2/Motor Out A: track 0.00 -> 60.0 mm
- net /Motor 1/Motor Out A: track 0.00 -> 58.6 mm
- net /Motor 2/Motor Out B: track 0.00 -> 13.7 mm
- net /Motor 3/Motor Out B: track 0.00 -> 13.6 mm
- net /Motor 4/Motor Out B: track 0.00 -> 13.6 mm
- net /Motor 1/Motor Out B: track 0.00 -> 13.5 mm
- net Net-(TP26-Pad1): track 0.00 -> 3.27 mm

Commit message: chore: l2
Parts:
- J17, J18, J3, J5: moved to B.Cu
- moved J12 36.4 mm to (42.5, 82.4), turned to 180 degrees
- moved J17 25.5 mm to (164.0, 129.2), turned to 180 degrees
- moved J18 24.0 mm to (68.0, 128.4), turned to 180 degrees
- moved KillSwitch2 21.1 mm to (43.0, 90.2), turned to 180 degrees
- moved U3 18.9 mm to (42.8, 110.2), turned to 90 degrees
- moved J5 14.6 mm to (137.0, 33.2), turned to 90 degrees
- moved TP28 13.3 mm to (198.3, 96.7), turned to 90 degrees
- moved TP1 9.06 mm to (198.3, 108.9), turned to 90 degrees
- moved J1 8.64 mm to (79.8, 144.7)
- moved J2 8.64 mm to (82.0, 151.7)
- moved TP3 8.40 mm to (198.3, 115.0), turned to 90 degrees
- moved R33 6.05 mm to (137.3, 36.9)
- moved J19 1.52 mm to (188.3, 124.7)
- moved J6 1.52 mm to (188.3, 118.7)
- moved J7 1.52 mm to (188.3, 130.7)
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Connections:
- J1 pad 2: /Dribbler Data -> /Dribbler PWM
- TP26 pad 1: Net-(TP26-Pad1) -> /Dribbler PWM
- TP27 pad 1: Net-(TP27-Pad1) -> /Sol
- U1 pad 12: Net-(TP26-Pad1) -> /Dribbler PWM
- U1 pad 13: Net-(TP27-Pad1) -> /Sol
Routing:
- net +12V: track 0.00 -> 30.7 mm
- net /Sol: track 0.00 -> 12.2 mm
- net Net-(J12-POS): track 0.00 -> 8.00 mm
- net Net-(TP26-Pad1): track 3.27 -> 0.00 mm
- net /Dribbler PWM: track 0.00 -> 3.27 mm
- net /Motors Enable: track 28.3 -> 30.3 mm
- added copper zone on F.Cu, net +12V
Other:
- board text added: "12v"
- board text added: "3v3"
- board text added: "5v"
- board text added: "Dribbler"
- board text added: "GND"
- board text added: "L1"
- board text added: "L3"
- board text added: "LIGHTGATE"
- board text added: "M-EN"
- board text added: "SOL"
- board text added: "Vent Exhaust"

Commit message: chore: l2
Parts:
- moved J18 2.25 mm to (68.0, 126.2)
- moved J17 1.75 mm to (164.0, 127.4)

Commit message: chore: l2
Parts:
- R33: moved to B.Cu
- turned R33 to 180 degrees
Routing:
- net +3V3: track 0.00 -> 504.0 mm, vias 0 -> 8
- net /Motors Enable: track 30.3 -> 175.5 mm, vias 0 -> 8
- net +12V: track 30.7 -> 123.3 mm, vias 0 -> 96
- net /Sol: track 12.2 -> 27.0 mm
- net Net-(TP25-Pad1): track 0.00 -> 3.08 mm
- net /RX (L3-Cam: track 0.00 -> 3.07 mm
- net /TX (L3-Teensy): track 0.00 -> 3.06 mm
- net /TX (L3-Cam): track 0.00 -> 3.06 mm
- net /RX (L3-Teensy): track 0.00 -> 3.05 mm
- net /TX (L1-Teensy): track 0.00 -> 3.04 mm
- net /SCL (IMU): track 0.00 -> 3.03 mm
- net Net-(TP24-Pad1): track 0.00 -> 3.03 mm
- net /RX (L1-Teensy): track 0.00 -> 3.02 mm
- net /SDA (IMU): track 0.00 -> 3.01 mm
- net /Motor 1 IN B: track 82.9 -> 85.7 mm
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- added copper zone on F.Cu, net +3V3
- added copper zone on F.Cu, net +5V
