File: elec/layer2/layer2.kicad_sch (KiCad schematic)
At the start: 0 parts

Commit message: fix: l1 gnd
Parts:
- added J1: Conn_01x03, Pinheaders:PinHeader_1x03_P2.54mm_Vertical, symbol Connector_Generic:Conn_01x03
- added J2: XT30UPB-M, layer2-pcb-footprints:AMASS_XT30UPB-M, symbol layer2-pcb-symbols:XT30UPB-M
- added SW1: SW_SPDT_312, layer2-pcb-footprints:SS12D00G3, symbol Switch:SW_SPDT_312
- added TP1, TP2: TestPoint_2Pole, TestPoint:TestPoint_2Pads_Pitch2.54mm_Drill0.8mm, symbol Connector:TestPoint_2Pole
- added U1: TEENSY40, layer2-pcb-footprints:TEENSY40, symbol layer2-pcb-symbols:TEENSY40
Connections:
- new net +12V: J2.P
- new net +3V3: J1.1 (Pin_1), SW1.3 (A), TP2.1
- new net +5V: TP1.1
- new net Dribbler Data: J1.2 (Pin_2)
- new net GND: J1.3 (Pin_3), J2.N, SW1.2 (C), TP1.2, TP2.2, U1.G1
- new net Motors Enable: SW1.1 (B)
- no-connect marks 0 -> 13
Other:
- added sheet Motor 1 (motor.kicad_sch)
- added sheet Motor 2 (motor.kicad_sch)
- added sheet Motor 3 (motor.kicad_sch)
- added sheet Motor 4 (motor.kicad_sch)
- note added: "Dribbler"
- note added: "MCU"
- note added: "Motors"
- note added: "Motors Enable"
- note added: "Testpoints"
- company: (none) -> Chen-Xuan Ng
- title: (none) -> A PCB

Commit message: fix: l1; chore: l2 schematics
Parts:
- added J3, J4: Conn_01x04, Connector_JST:JST_XH_B4B-XH-AM_1x04_P2.50mm_Vertical, symbol Connector_Generic:Conn_01x04
- added J5: Conn_01x03, Pinheaders:PinHeader_1x03_P2.54mm_Vertical, symbol Connector_Generic:Conn_01x03
- added J6, J7, J8, J9: XT30PW-M, layer1-pcb-footprints:AMASS_XT30PW-M, symbol layer1-pcb-symbols:XT30PW-M
- added R33: 10k, symbol Device:R
Connections:
- net +12V: now also J8.P
- net +3V3: now also J5.1 (Pin_1), J6.P, J9.P
- net +5V: now also U1.VIN, J7.P
- net GND: now also U1.G2, U1.G3, J3.1 (Pin_1), J3.4 (Pin_4), J4.1 (Pin_1), J4.4 (Pin_4), J5.3 (Pin_3), J6.N, J7.N, J8.N, J9.N, R33.2
- net Motor 1 IN A: now also U1.4
- net Motor 1 IN B: now also U1.5
- net Motor 1 PWM: now also U1.0
- net Motor 2 IN A: now also U1.6
- net Motor 2 IN B: now also U1.7
- net Motor 2 PWM: now also U1.1
- net Motor 3 IN A: now also U1.8
- net Motor 3 IN B: now also U1.9
- net Motor 3 PWM: now also U1.2
- net Motor 4 IN A: now also U1.10
- net Motor 4 IN B: now also U1.11
- net Motor 4 PWM: now also U1.3
- net TX (L1-Teensy): now reaches U1.16
- net TX (L1-Teensy): now also J3.3 (Pin_3)
- net RX (L1-Teensy): now reaches U1.17
- net RX (L1-Teensy): now also J3.2 (Pin_2)
- net RX (L3-Teensy): now reaches U1.20
- net RX (L3-Teensy): now also J4.2 (Pin_2)
- net TX (L3-Teensy): now reaches U1.21
- net TX (L3-Teensy): now also J4.3 (Pin_3)
- new net Sol: J5.2 (Pin_2), R33.1
- no-connect marks 13 -> 1
Other:
- note added: "Batt"
- note added: "Kicker"
- note added: "Layer-to-Layer Communication"
- note added: "Layer1"
- note added: "Layer1 Power"
- note added: "Layer2 Power"
- note added: "Layer3"
- note added: "Power"
- moved on the sheet: J1, J2, SW1, TP1, TP2, U1

Commit message: feat: l2 schematics
Parts:
- removed J4: Conn_01x04, Connector_JST:JST_XH_B4B-XH-AM_1x04_P2.50mm_Vertical, symbol Connector_Generic:Conn_01x04
- added H1, H10, H11, H12, H2, H3, H4, H5, H6, H7, H8, H9: MountingHole, symbol Mechanical:MountingHole
- added J10, J11, J4: Conn_01x05, symbol Connector_Generic:Conn_01x05
- added J12: XT60-M, layer2-pcb-footprints:AMASS_XT60-M, symbol layer2-pcb-symbols:XT60-M
- added J17, J18: Conn_01x02, symbol Connector_Generic:Conn_01x02
- added KillSwitch2: SW_SPST, Connector_AMASS:AMASS_XT30U-F_1x02_P5.0mm_Vertical, symbol Switch:SW_SPST
- added TP16, TP17, TP18, TP19, TP20, TP21, TP22, TP23, TP24, TP25, TP26, TP27: TestPoint, symbol Connector:TestPoint
- added TP3: TestPoint_2Pole, TestPoint:TestPoint_2Pads_Pitch2.54mm_Drill0.8mm, symbol Connector:TestPoint_2Pole
Connections:
- net +12V: now also KillSwitch2.1 (A), TP3.1
- net +3V3: now also J17.1 (Pin_1), J18.1 (Pin_1)
- net GND: now also J10.5 (Pin_5), J11.5 (Pin_5), J12.N (NEG), J17.2 (Pin_2), J4.5 (Pin_5), TP3.2
- net RX (L1-Teensy): now also TP20.1
- net RX (L3-Teensy): now also J4.1 (Pin_1), TP17.1
- net TX (L1-Teensy): now also TP21.1
- net TX (L3-Teensy): now also J4.2 (Pin_2), TP16.1
- net at U1.12: now also TP26.1
- net at U1.13: now also TP27.1
- net RX (L3-Cam: now reaches U1.14
- net RX (L3-Cam: now also J4.3 (Pin_3), TP23.1
- net TX (L3-Cam): now reaches U1.15
- net TX (L3-Cam): now also J4.4 (Pin_4), TP22.1
- net SDA (IMU): now reaches U1.18
- net SDA (IMU): now also J10.2 (Pin_2), TP19.1
- net SCL (IMU): now reaches U1.19
- net SCL (IMU): now also J10.1 (Pin_1), TP18.1
- net at U1.22: now also TP25.1
- net at U1.23: now also TP24.1
- new net: J12.P (POS), KillSwitch2.2 (B)
- new net Lightgate: J18.2 (Pin_2)
- new net SW (1): J11.1 (Pin_1)
- new net SW (2): J11.2 (Pin_2)
- new net SW (3): J11.3 (Pin_3)
- new net SW (4): J11.4 (Pin_4)
- new net SW (GOAL): J10.3 (Pin_3)
- new net SW (ROLE): J10.4 (Pin_4)
- no-connect marks 1 -> 5
Other:
- note added: "Layer3 Power"
- note added: "Lightgate"
- note added: "Mounting Holes"
- note removed: "Layer2 Power"
- moved on the sheet: J3, J7, J8, TP1, TP2

Commit message: feat: buck.steps; chore: l2
Parts:
- added TP28: TestPoint_2Pole, TestPoint:TestPoint_2Pads_Pitch2.54mm_Drill0.8mm, symbol Connector:TestPoint_2Pole
- added U3: ~, layer2-pcb-footprints:buck-module, symbol layer2-pcb-symbols:buck-module
- H1, H10, H11, H12, H2, H3, H4, H5, H6, H7, H8, H9: footprint (none) -> MountingHole:MountingHole_3.2mm_M3_DIN965_Pad
- J1, J5: footprint Pinheaders:PinHeader_1x03_P2.54mm_Vertical -> Connector_JST:JST_XH_B3B-XH-A_1x03_P2.50mm_Vertical
- J10, J11, J4: footprint (none) -> Connector_JST:JST_XH_B5B-XH-A_1x05_P2.50mm_Vertical
- J17, J18: footprint (none) -> Connector_JST:JST_XH_B2B-XH-A_1x02_P2.50mm_Vertical
- J3: footprint Connector_JST:JST_XH_B4B-XH-AM_1x04_P2.50mm_Vertical -> Connector_JST:JST_XH_B4B-XH-A_1x04_P2.50mm_Vertical
- J6, J7, J8, J9: footprint layer1-pcb-footprints:AMASS_XT30PW-M -> layer2-pcb-footprints:AMASS_XT30PW-M
- KillSwitch2: footprint Connector_AMASS:AMASS_XT30U-F_1x02_P5.0mm_Vertical -> layer2-pcb-footprints:AMASS_XT30UPB-M
- R33: footprint (none) -> Resistor_SMD:R_0603_1608Metric
- TP16, TP17, TP18, TP19, TP20, TP21, TP22, TP23, TP24, TP25, TP26, TP27: footprint (none) -> TestPoint:TestPoint_THTPad_D1.5mm_Drill0.7mm
Connections:
- net +12V: now also KillSwitch2.N (A), U3.1 (12v); no longer KillSwitch2.1 (A)
- net +3V3: now also U3.4 (3v3)
- net +5V: now also U3.3 (5v)
- net GND: now also TP28.1, TP28.2, U3.2 (GND)
- net Motor 1 IN A: now also U1.0; no longer U1.4
- net Motor 1 IN B: now also U1.2; no longer U1.5
- net Motor 1 PWM: now also U1.1; no longer U1.0
- net Motor 2 IN A: now also U1.3; no longer U1.6
- net Motor 2 IN B: now also U1.5; no longer U1.7
- net Motor 2 PWM: now also U1.4; no longer U1.1
- net Motor 3 IN A: now also U1.6; no longer U1.8
- net Motor 3 IN B: now also U1.8; no longer U1.9
- net Motor 3 PWM: now also U1.7; no longer U1.2
- net Motor 4 IN A: now also U1.9; no longer U1.10
- net Motor 4 PWM: now also U1.10; no longer U1.3
- net at J12.P (POS): now also KillSwitch2.P (B); no longer KillSwitch2.2 (B)
Other:
- moved on the sheet: TP1, TP2, TP3

Commit message: chore: l2
Parts:
- removed J6, J7, J8: XT30PW-M, layer2-pcb-footprints:AMASS_XT30PW-M, symbol layer1-pcb-symbols:XT30PW-M
- added J19, J6, J7: XT30UPB-M, layer2-pcb-footprints:AMASS_XT30UPB-M, symbol layer2-pcb-symbols:XT30UPB-M
Connections:
- net +12V: now also J7.P
- net +3V3: now also J19.P
- net +5V: now also J6.P
- net GND: now also J19.N, J6.N, J7.N

Commit message: chore: l2
Connections:
- net Dribbler Data is gone; now on net Dribbler PWM: J1.2 (Pin_2)
- net Sol: now also TP27.1, U1.13
- net Dribbler PWM: now reaches TP26.1, U1.12
Other:
- moved on the sheet: TP26
Changed lines of the file:
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@@
-	(wire
-		(pts
-			(xy 207.01 81.28) (xy 219.71 81.28)
-		)
-		(stroke
-			(width 0)
-			(type default)
-		)
-	)
 	(wire
 		(pts
@@
 		(pts
 			(xy 355.6 99.06) (xy 355.6 97.79)
+		)
+		(stroke
+			(width 0)
+			(type default)
+		)
+	)
+	(wire
+		(pts
+			(xy 205.74 81.28) (xy 219.71 81.28)
 		)
 		(stroke
@@
 		)
 	)
-	(label "Dribbler Data"
+	(label "Dribbler PWM"
 		(at 31.75 64.77 0)
 		(effects
@@
 		)
 	)
+	(label "Dribbler PWM"
+		(at 205.74 81.28 0)
+		(effects
+			(font
+				(size 1.27 1.27)
+			)
+			(justify left bottom)
+		)
+	)
 	(label "Motor 2 IN A"
 		(at 205.74 58.42 0)
@@
 	(label "Motor 1 PWM"
 		(at 90.17 163.83 180)
+		(effects
+			(font
+				(size 1.27 1.27)
+			)
+			(justify right bottom)
+		)
+	)
+	(label "Sol"
+		(at 271.78 81.28 180)
 		(effects
 			(font
@@
 	(symbol
 		(lib_id "Connector:TestPoint")
-		(at 207.01 81.28 90)
+		(at 205.74 81.28 90)
 		(unit 1)
 		(exclude_from_sim no)
@@
 		(dnp no)
 		(property "Reference" "TP26"
-			(at 197.612 80.01 90)
+			(at 196.342 80.01 90)
 			(effects
 				(font
@@
 		)
 		(property "Value" "TestPoint"
-			(at 197.612 82.55 90)
+			(at 196.342 82.55 90)
 			(effects
 				(font
@@
 		)
 		(property "Footprint" "TestPoint:TestPoint_THTPad_D1.5mm_Drill0.7mm"
-			(at 207.01 76.2 0)
+			(at 205.74 76.2 0)
 			(effects
 				(font
@@
 		)
 		(property "Datasheet" "~"
-			(at 207.01 76.2 0)
+			(at 205.74 76.2 0)
 			(effects
 				(font
@@
 		)
 		(property "Description" "test point"
-			(at 207.01 81.28 0)
-			(effects
-				(font
+			(at 205.74 81.28 0)
+			(effects
+				(font

Commit message: prod: prod
Parts:
- R33: value 10k -> 10K
Changed lines of the file:
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@@
 			)
 		)
-		(property "Value" "10k"
+		(property "Value" "10K"
 			(at 128.27 69.8499 0)
 			(effects

Commit message: fix: l2
Parts:
- removed J11: Conn_01x05, Connector_JST:JST_XH_B5B-XH-A_1x05_P2.50mm_Vertical, symbol Connector_Generic:Conn_01x05
- added TP29, TP30, TP31: TestPoint, TestPoint:TestPoint_THTPad_D1.5mm_Drill0.7mm, symbol Connector:TestPoint
Connections:
- net +5V: now also TP30.1
- net GND: now also TP31.1
- net Lightgate: now also TP25.1, U1.22
- net at U1.3.3V_2: now also TP29.1
- net SW (GOAL): no longer names the net of J10.3 (Pin_3)
- net SW (ROLE): no longer names the net of J10.4 (Pin_4)
- no-connect marks 5 -> 6
Other:
- moved on the sheet: J10, J3, J4
